File: projects/RADIO/SA612_RCVR/Sa612_RCVR/sa612_rcvr.brd (EAGLE design)
At the start: 60 x 40 mm, 39 parts, among them IC1 SA612AN, Q1 BC238

Commit message: update
Parts:
- C7: device rcl:C050-050X075 -> rcl:C050-025X075
- TR1: value 71K-5412 -> 71K-1524
- moved C2 3.32 mm to (15.4, 23.4)
- moved C1 1.71 mm to (24.5, 31.8)
- moved R5 1.56 mm to (31.7, 4.01)
- moved C6 0.50 mm to (41.8, 31.7)
- moved U$4 0.48 mm to (5.39, 19.1)
- moved U$3 0.45 mm to (5.39, 22.5)
- moved TR1 0.41 mm to (16.6, 31.6), turned to 90 degrees
- moved C7 0.36 mm to (47.7, 32.0), flipped to the top
- moved C1-1 0.34 mm to (22.4, 31.8), flipped to the top
- moved C11 0.14 mm to (32.3, 19.4)
- moved C13 0.10 mm to (25.6, 19.4)
Connections:
- net ANTENA: now also TR1.4; no longer TR1.2
- net GND: now also TR1.2; no longer TR1.1
- net N$1: now also TR1.5; no longer TR1.4
- net N$2: now also TR1.1; no longer TR1.5
Routing:
- net N$12: track 43.6 -> 48.6 mm
- net N$2: track 18.6 -> 22.1 mm
- net GND: track 0.00 -> 2.71 mm
- net N$13: track 27.8 -> 29.8 mm
- net N$10: track 7.77 -> 8.59 mm
- net N$5: track 7.49 -> 8.19 mm
- net N$1: track 10.5 -> 9.79 mm
- net OUT: track 5.11 -> 5.72 mm
- net ANTENA: track 17.7 -> 18.2 mm
- net N$6: track 8.73 -> 9.23 mm
