File: projects/RADIO/2-SA612_RCVR/2-sa612_rcvr/mixer_bolock.brd (EAGLE design)
At the start: 75 x 45 mm, 29 parts, among them IC1 SA612AN_01,112, IC2 SA612AN_01,112

Commit message: update
Parts:
- C1, C2, C3, C7, C8: value 10pF -> 10nF
