File: projects/RADIO/SA612_LM386/sa612_lm386/sa612_lm386.brd (EAGLE design)
At the start: 75 x 45 mm, 29 parts, among them IC1 SA612AN_01,112, IC2 SA612AN_01,112

Commit message: update
Parts:
- removed +5, BFI, IN, U$2, U$4, U$5, U$6, U$7, VFI: SMD_PIN, mylib:SMD_PIN
- removed U$1: ZTBF455E, mylib:ZTBF455E
- removed U$9: LT455EU, mylib:LT455EU
- added C11: 100pF, mylib:C0805K
- added C12, C13: 100nF, mylib:C0805
- added C14: 10uF, mylib:E5-5
- added CON_1, CON_2, RF_IN: 2X_SMD_PTH_PIN, mylib:2X_SMD_PTH
- added IC3: LM1117MPX-33NOPB, LM1117MPX-33NOPB:SOT230P700X180-4N
- added IN_A, IN_B, P_1: SMD_PIN, mylib:SMD_PIN
- added L1: 10uH, mylib:M0805
- added LED_1: (no value), mylib:CHIP-LED0805
- added Q1: BF245, transistor-fet:TO92
- added R2, R3: (no value), mylib:R0805W
- added R4, R5: 10k, mylib:R0805W
- added R6: (no value), mylib:R0805
- added R7: 1M, mylib:R0805
- added R8: 100, mylib:R0805W
- added R9: (no value), rcl:RTRIM64W
- C1, C8: value 10pF -> 10nF; device rcl:C0805K -> mylib:C0805
- C10: value 100nF -> 33nF; device rcl:C0805K -> mylib:C0805K
- C2, C3: value 10pF -> 20nF; device rcl:C0805K -> mylib:C0805K
- C4: value 470pF -> 33nF; device rcl:C0805K -> mylib:C0805K
- C5: value 470pF -> 10uF; device rcl:C0805K -> mylib:E5-5
- C6: value 2.2uF -> 10nF; device rcl:C050-050X075 -> mylib:C0805
- C7: value 10pF -> 47uF; device rcl:C0805K -> mylib:E5-5
- C9: value 100nF -> 10nF; device rcl:C0805K -> mylib:C0805
- IC2: value SA612AN_01,112 -> LM386M-1; device SA612AN_01_112:DIP762W53P254L950H420Q8N -> linear:SO08
- OUT: value SMD_PIN -> 2X_SMD_PTH_PIN; device mylib:SMD_PIN -> mylib:2X_SMD_PTH
- R1: value 470R -> (none); device rcl:R0805 -> mylib:R0805
- moved C10 44.2 mm to (12.5, 12.0), turned to 0 degrees
- moved R1 40.9 mm to (12.5, 16.0), turned to 180 degrees
- moved C6 35.5 mm to (67.2, 16.8), turned to 90 degrees
- moved C7 33.7 mm to (64.3, 16.5), turned to 270 degrees
- moved C9 30.7 mm to (22.4, 23.2), turned to 0 degrees
- moved OUT 30.2 mm to (48.0, 6.50)
- moved C1 25.6 mm to (37.5, 36.4), turned to 270 degrees
- moved C5 24.6 mm to (58.5, 27.7), flipped to the bottom
- moved IC2 21.5 mm to (58.3, 22.1), flipped to the top, turned to 270 degrees
- moved C8 19.3 mm to (56.2, 16.6)
- moved C4 18.7 mm to (37.5, 22.0), turned to 90 degrees
- moved IC1 14.3 mm to (30.0, 22.0), turned to 270 degrees
- moved C3 11.7 mm to (47.5, 25.0), turned to 180 degrees
- moved C2 7.81 mm to (47.5, 19.0)
- moved H3 5.00 mm to (15.0, 44.0)
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Connections:
- removed net BFI: BFI.P$1, C4.2, C5.1, IC2.6, U$1.P$1
- removed net OUT: C6.2, OUT.P$1
- removed net RF_INPUT: IC1.1, IN.P$1
- removed net VFI: R1.2, VFI.P$1
- new net 12V: C14.-, CON_2.P$1, CON_2.T$1, IC3.3, R6.1, R6.P$1, R8.1
- new net N$13: C6.2, R4.1
- new net N$14: C6.1, C7.-, LED_1.C, LED_1.CP, OUT.P$1, OUT.T$1
- new net N$15: C7.+, IC2.5, R5.1
- new net N$16: C8.1, R5.2
- new net N$17: C10.2, C10.P$2, Q1.2, R1.1, R1.P$1
- new net N$18: C9.1, Q1.1, R6.2, R6.P$2
- new net N$19: C11.2, C11.P$2, Q1.3, R7.1, R7.P$1
- new net N$2: C1.2, IC1.2, IN_B.P$1, L1.1, L1.P$1, LED_1.A, LED_1.AP
- new net N$20: C11.1, C11.P$1, RF_IN.P$1, RF_IN.T$1
- new net N$21: C13.2, IC2.6, R8.2
- new net N$22: CON_1.P$1, CON_1.T$1, R9.2
- new net N$7: C4.1, C4.P$1, IC1.5, R2.2
- new net N$9: IC1.6, R9.1
- net 5V: now also C12.2, IC3.2, IC3.4; no longer +5.P$1, C10.1, C9.1, IC2.8
- net GND: now also C10.1, C10.P$1, C12.1, C13.1, C14.+, C8.2, CON_1.P$2, CON_1.T$2, CON_2.P$2, CON_2.T$2, IC2.4, IC3.1, OUT.P$2, OUT.T$2, R1.2, R1.P$2, R7.2, R7.P$2, R9.3, RF_IN.P$2, RF_IN.T$2; no longer C10.2, C2.1, C5.2, C7.1, C8.1, C9.2, IC2.3, U$1.P$2, U$2.P$1, U$4.P$1, U$5.P$1, U$6.P$1, U$7.P$1, U$9.GND
- net N$1: now also C9.2, IC1.1, IN_A.P$1, L1.2, L1.P$2; no longer C1.2, IC1.2
- net N$10: now also IC1.7, P_1.P$1; no longer C6.1, C7.2, IC2.4
- net N$11: now also C5.+, IC2.1; no longer C8.2, IC2.2
- net N$12: now also C5.-, IC2.8, R4.2; no longer IC1.5, U$9.IN
- net N$3: now also C2.1, C2.P$1, IC2.3; no longer IC2.1, U$9.OUT
- net N$4: now also C3.1, C3.P$1, IC2.2; no longer C2.2, IC1.4
- net N$5: now also C3.P$2, R3.1; no longer R1.1
- net N$6: now also C2.2, C2.P$2, R2.1; no longer C3.1, IC1.6
- net N$8: now also C4.2, C4.P$2, IC1.4, R3.2; no longer C4.1, IC2.7
Routing:
- net N$14: track 0.00 -> 57.6 mm, vias 0 -> 2
- net 12V: track 0.00 -> 56.8 mm
- net BFI: track 35.4 -> 0.00 mm
- net N$2: track 0.00 -> 25.3 mm
- net N$21: track 0.00 -> 17.7 mm
- net 5V: track 49.6 -> 64.9 mm
- net N$1: track 2.81 -> 16.9 mm
- net N$17: track 0.00 -> 13.1 mm
- net OUT: track 12.5 -> 0.00 mm
- net N$19: track 0.00 -> 11.7 mm
- net N$18: track 0.00 -> 9.93 mm
- net N$7: track 0.00 -> 8.13 mm
- net N$20: track 0.00 -> 7.50 mm
- net N$15: track 0.00 -> 6.63 mm
- net N$9: track 0.00 -> 6.29 mm
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Other:
- board size 75 x 45 mm -> 75 x 50 mm

Commit message: update
Parts:
- removed R3: (no value), mylib:R0805W
- added C15: 47nF, mylib:C0805
- added C16: 1nF, mylib:C0805
- C2, C3: value 20nF -> 100nF
- C4: value 33nF -> 47nF
- R1: value (none) -> 1k
- R2, R6: value (none) -> 4k7
- moved C3 3.50 mm to (44.0, 25.0)
- moved OUT 1.13 mm to (48.2, 5.40)
- moved C11 1.00 mm to (11.5, 27.0)
- moved CON_1 1.00 mm to (35.5, 5.50)
- moved P_1 1.00 mm to (30.1, 5.50)
- moved C2 0.50 mm to (47.0, 19.0)
- moved R9 0.50 mm to (33.8, 12.7)
- moved R2 0.45 mm to (40.7, 19.0)
- moved CON_2 0.22 mm to (9.60, 34.7)
Connections:
- net N$3: now also C15.1
- net N$4: now also C15.2
- net N$5: now also C16.2, R9.1; no longer C3.2, C3.P$2, R3.1
- net N$8: now also C3.2, C3.P$2; no longer R3.2
- net N$9: now also C16.1; no longer R9.1
Routing:
- net N$4: track 7.84 -> 12.7 mm
- net N$9: track 6.29 -> 2.50 mm
- net N$3: track 7.89 -> 10.5 mm
- net 5V: track 64.9 -> 67.1 mm
- net N$5: track 3.80 -> 1.81 mm
- net N$8: track 8.13 -> 9.23 mm
- net N$20: track 7.50 -> 6.50 mm
- net N$19: track 11.7 -> 10.7 mm
- net N$10: track 12.3 -> 13.3 mm
- net N$14: track 57.6 -> 58.6 mm
- net N$22: track 3.06 -> 3.56 mm

Commit message: update
Parts:
- removed R9: (no value), rcl:RTRIM64W
- added C17: 1nF, mylib:C0805
- added L2: 10uH, mylib:M0805
- added R3: 51R, mylib:R0805W
- moved C14 6.58 mm to (37.0, 39.1)
- moved C1 4.36 mm to (41.9, 36.0), turned to 180 degrees
- moved CON_1 4.00 mm to (39.5, 5.50)
- moved C13 3.80 mm to (63.6, 34.8), turned to 270 degrees
- moved C5 1.80 mm to (59.5, 29.2)
- moved IC2 1.80 mm to (59.3, 23.6)
- moved R4 1.80 mm to (68.2, 24.2)
- moved C16 1.70 mm to (31.3, 16.1)
- moved C15 1.50 mm to (50.0, 23.9)
- moved C2 1.50 mm to (47.0, 20.5)
- moved C3 1.50 mm to (44.0, 26.5)
- moved C4 1.50 mm to (37.5, 23.5)
- moved IC1 1.50 mm to (30.0, 23.5)
- moved OUT 1.50 mm to (49.8, 5.40)
- moved R2 1.50 mm to (40.7, 20.5)
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Connections:
- new net N$23: C17.2, L2.1, L2.P$1
- net GND: now also R3.1; no longer R9.3
- net N$22: now also C17.1; no longer R9.2
- net N$5: now also L2.2, L2.P$2, R3.2; no longer R9.1
Routing:
- net N$5: track 1.81 -> 8.25 mm
- net N$23: track 0.00 -> 4.60 mm
- net 5V: track 67.1 -> 69.6 mm
- net GND: track 4.75 -> 2.70 mm
- net 12V: track 56.6 -> 58.4 mm
- net N$2: track 25.3 -> 26.9 mm
- net N$10: track 13.3 -> 14.8 mm
- net N$12: track 10.2 -> 11.5 mm
- net N$4: track 12.7 -> 13.7 mm
- net N$3: track 10.5 -> 11.5 mm
- net N$17: track 13.1 -> 12.1 mm
- net N$1: track 17.2 -> 16.2 mm
- net N$13: track 3.50 -> 4.22 mm
- net N$21: track 17.7 -> 17.1 mm
- net N$20: track 6.50 -> 7.00 mm
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
Commit message: Update
Parts:
- removed R4: 10k, mylib:R0805W
- added C18: 10uF, mylib:E5-5
- added R9: (no value), rcl:RTRIM64W
- moved C12 17.9 mm to (32.1, 26.9), turned to 180 degrees
- moved C13 13.9 mm to (58.6, 21.8), turned to 0 degrees
- moved C14 13.9 mm to (49.9, 44.3), turned to 270 degrees
- moved IC3 12.5 mm to (39.5, 48.0)
- moved P_1 8.47 mm to (26.2, 13.1)
- moved R5 8.13 mm to (55.1, 18.1)
- moved R3 7.98 mm to (31.4, 12.8), turned to 90 degrees
- moved C8 7.49 mm to (48.9, 18.1)
- moved C5 7.26 mm to (59.8, 36.5)
- moved C17 7.15 mm to (38.0, 12.9)
- moved R8 6.02 mm to (59.8, 40.8)
- moved CON_2 5.47 mm to (10.5, 40.1)
- moved H3 5.00 mm to (15.0, 49.0)
- moved H4 5.00 mm to (60.0, 49.0)
- moved L2 4.91 mm to (36.9, 17.9), turned to 180 degrees
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Connections:
- net 5V: now also C18.+
- net GND: now also C18.-
- net N$12: now also R9.3; no longer R4.2
- net N$13: now also R9.1, R9.2; no longer R4.1
Routing:
- net N$15: track 7.13 -> 13.7 mm
- net 5V: track 69.6 -> 65.8 mm
- net N$14: track 58.7 -> 62.3 mm
- net N$21: track 17.1 -> 20.4 mm
- net N$19: track 11.2 -> 14.4 mm
- net N$11: track 3.84 -> 7.01 mm
- net N$17: track 12.1 -> 15.3 mm
- net N$10: track 14.8 -> 11.7 mm
- net N$13: track 4.22 -> 6.53 mm
- net 12V: track 58.4 -> 56.4 mm
- net N$8: track 9.23 -> 11.2 mm
- net N$18: track 10.4 -> 11.7 mm
- net N$4: track 13.7 -> 15.0 mm
- net N$3: track 11.5 -> 12.6 mm
- net N$9: track 2.30 -> 3.30 mm
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Other:
- board size 75 x 50 mm -> 75 x 55 mm

Commit message: Update 07/06/2022
Routing:
- net 12V: track 56.4 -> 57.0 mm
