File: projects/RADIO/SA612_LM386/sa612_lm386/sa612_lm386.sch (EAGLE design)
At the start: 40 parts, among them IC1 SA612AN_01,112, IC2 LM386M-1, IC3 LM1117MPX-33NOPB, Q1 BF245

Commit message: update
Parts:
- removed R3: (no value), mylib:R_0805_SMD
- added C15: 47nF, mylib:C_0805_SMD
- added C16: 1nF, mylib:C_0805_SMD
- C2, C3: value 20nF -> 100nF
- C4: value 33nF -> 47nF
- R1: value (none) -> 1k
- R2, R6: value (none) -> 4k7
Connections:
- net N$3: now also C15.1
- net N$4: now also C15.2
- net N$5: now also C16.2, R9.A; no longer C3.2, R3.1
- net N$8: now also C3.2; no longer R3.2
- net N$9: now also C16.1; no longer R9.A
Other:
- moved on the sheet: C2, C3, C4, CON_1, R2, R9

Commit message: update
Parts:
- removed R9: (no value), rcl:R-TRIMM64W
- added C17: 1nF, mylib:C_0805_SMD
- added L2: 10uH, mylib:L_0805_PTH
- added R3: 51R, mylib:R_0805_SMD
Connections:
- new net N$23: C17.2, L2.1
- net GND: now also R3.1; no longer R9.E
- net N$22: now also C17.1; no longer R9.S
- net N$5: now also L2.2, R3.2; no longer R9.A
Other:
- moved on the sheet: CON_1

Commit message: Update
Parts:
- removed R4: 10k, mylib:R_0805_SMD
- added C18: 10uF, mylib:C_POL
- added R9: (no value), rcl:R-TRIMM64W
Connections:
- net 5V: now also C18.+
- net GND: now also C18.-
- net N$12: now also R9.E; no longer R4.2
- net N$13: now also R9.A, R9.S; no longer R4.1
