File: projects/RADIO/fq_divider/divider.sch (EAGLE design)
At the start: 13 parts, among them IC1 SN74AC74D

Commit message: Update
Parts:
- removed RX_CLK0, RX_CLK1: SMD_PTH_PIN, mylib:SMD_PTH_PIN
- added H3, H4: MOUNT-PAD-ROUND2.8, holes:MOUNT-PAD-ROUND2.8
- added QSD_CLK0, QSD_CLK1: 2X_SMD_PTH_PIN, mylib:2X_SMD_PTH_PIN
Connections:
- net GND: now also H3.MOUNT, H4.MOUNT, QSD_CLK0.PIN1, QSD_CLK1.PIN0
- net QSD_CLK0: now also QSD_CLK0.PIN0; no longer RX_CLK0.P$1
- net QSD_CLK1: now also QSD_CLK1.PIN1; no longer RX_CLK1.P$1
Changed lines of the file:
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@@
 <part name="SUPPLY4" library="SparkFun-PowerSymbols" deviceset="VCC" device=""/>
 <part name="GND2" library="SparkFun-PowerSymbols" deviceset="GND" device=""/>
-<part name="RX_CLK1" library="mylib" deviceset="SMD_PTH_PIN" device=""/>
-<part name="RX_CLK0" library="mylib" deviceset="SMD_PTH_PIN" device=""/>
 <part name="TX_CLK0" library="mylib" deviceset="SMD_PTH_PIN" device=""/>
 <part name="TX_CLK1" library="mylib" deviceset="SMD_PTH_PIN" device=""/>
@@
 <part name="SUPPLY5" library="SparkFun-PowerSymbols" deviceset="VCC" device=""/>
 <part name="GND7" library="SparkFun-PowerSymbols" deviceset="GND" device=""/>
+<part name="QSD_CLK1" library="mylib" deviceset="2X_SMD_PTH_PIN" device=""/>
+<part name="QSD_CLK0" library="mylib" deviceset="2X_SMD_PTH_PIN" device=""/>
+<part name="GND8" library="SparkFun-PowerSymbols" deviceset="GND" device=""/>
+<part name="H3" library="holes" library_urn="urn:adsk.eagle:library:237" deviceset="MOUNT-PAD-ROUND" device="2.8" package3d_urn="urn:adsk.eagle:package:14281/1"/>
+<part name="H4" library="holes" library_urn="urn:adsk.eagle:library:237" deviceset="MOUNT-PAD-ROUND" device="2.8" package3d_urn="urn:adsk.eagle:package:14281/1"/>
+<part name="GND9" library="SparkFun-PowerSymbols" deviceset="GND" device=""/>
+<part name="GND10" library="SparkFun-PowerSymbols" deviceset="GND" device=""/>
 </parts>
 <sheets>
@@
 <attribute name="VALUE" x="20.32" y="27.686" size="1.778" layer="96" align="top-center"/>
 </instance>
-<instance part="RX_CLK1" gate="G$1" x="68.58" y="5.08" smashed="yes" rot="R270"/>
-<instance part="RX_CLK0" gate="G$1" x="81.28" y="5.08" smashed="yes" rot="R270"/>
 <instance part="TX_CLK0" gate="G$1" x="43.18" y="5.08" smashed="yes" rot="R270"/>
 <instance part="TX_CLK1" gate="G$1" x="104.14" y="5.08" smashed="yes" rot="R270"/>
@@
 <instance part="GND7" gate="1" x="91.44" y="73.66" smashed="yes">
 <attribute name="VALUE" x="91.44" y="73.406" size="1.778" layer="96" align="top-center"/>
+</instance>
+<instance part="QSD_CLK1" gate="G$1" x="68.58" y="-10.16" smashed="yes" rot="R270">
+<attribute name="NAME" x="74.68" y="-11.24" size="1.27" layer="95" rot="R270"/>
+</instance>
+<instance part="QSD_CLK0" gate="G$1" x="78.74" y="-10.16" smashed="yes" rot="R270">
+<attribute name="NAME" x="84.84" y="-11.24" size="1.27" layer="95" rot="R270"/>
+</instance>
+<instance part="GND8" gate="1" x="75.184" y="-1.016" smashed="yes" rot="R180">
+<attribute name="VALUE" x="75.184" y="-0.762" size="1.778" layer="96" rot="R180" align="top-center"/>
+</instance>
+<instance part="H3" gate="G$1" x="66.04" y="93.98" smashed="yes">
+<attribute name="NAME" x="68.834" y="94.5642" size="1.778" layer="95"/>
+</instance>
+<instance part="H4" gate="G$1" x="66.04" y="101.6" smashed="yes">
+<attribute name="NAME" x="68.834" y="102.1842" size="1.778" layer="95"/>
+</instance>
+<instance part="GND9" gate="1" x="55.88" y="93.98" smashed="yes" rot="R270">
+<attribute name="VALUE" x="55.626" y="93.98" size="1.778" layer="96" rot="R270" align="top-center"/>
+</instance>
+<instance part="GND10" gate="1" x="55.88" y="101.6" smashed="yes" rot="R270">
+<attribute name="VALUE" x="55.626" y="101.6" size="1.778" layer="96" rot="R270" align="top-center"/>
 </instance>
 </instances>
@@
 <wire x1="86.28" y1="80.82" x2="91.44" y2="80.82" width="0.1524" layer="91"/>
 <wire x1="91.44" y1="80.82" x2="91.44" y2="76.2" width="0.1524" layer="91"/>
+</segment>
+<segment>
+<pinref part="QSD_CLK1" gate="G$1" pin="PIN0"/>
+<wire x1="71.58" y1="-7.7" x2="71.58" y2="-5.842" width="0.1524" layer="91"/>
+<wire x1="71.58" y1="-5.842" x2="75.184" y2="-5.842" width="0.1524" layer="91"/>
+<pinref part="QSD_CLK0" gate="G$1" pin="PIN1"/>
+<wire x1="75.184" y1="-5.842" x2="78.486" y2="-5.842" width="0.1524" layer="91"/>
+<wire x1="78.486" y1="-5.842" x2="78.74" y2="-5.842" width="0.1524" layer="91"/>
+<wire x1="78.74" y1="-5.842" x2="78.74" y2="-7.7" width="0.1524" layer="91"/>
+<pinref part="GND8" gate="1" pin="GND"/>
+<wire x1="75.184" y1="-3.556" x2="75.184" y2="-5.842" width="0.1524" layer="91"/>
+<junction x="75.184" y="-5.842"/>
+</segment>
+<segment>
+<pinref part="H3" gate="G$1" pin="MOUNT"/>
+<pinref part="GND9" gate="1" pin="GND"/>
+<wire x1="58.42" y1="93.98" x2="63.5" y2="93.98" width="0.1524" layer="91"/>
+</segment>
+<segment>
+<pinref part="H4" gate="G$1" pin="MOUNT"/>
+<pinref part="GND10" gate="1" pin="GND"/>
+<wire x1="58.42" y1="101.6" x2="63.5" y2="101.6" width="0.1524" layer="91"/>
 </segment>
 </net>
@@
 <junction x="68.58" y="20.32"/>
 <label x="73.66" y="-2.54" size="1.778" layer="95" rot="R90"/>
-<pinref part="RX_CLK1" gate="G$1" pin="P$1"/>
 <wire x1="68.58" y1="5.08" x2="68.58" y2="7.62" width="0.1524" layer="91"/>
+<pinref part="QSD_CLK1" gate="G$1" pin="PIN1"/>
+<wire x1="68.58" y1="-7.7" x2="68.58" y2="5.08" width="0.1524" layer="91"/>
 </segment>
 </net>
@@
 <pinref part="IC1" gate="G$1" pin="2D"/>
 <wire x1="96.52" y1="50.8" x2="83.82" y2="50.8" width="0.1524" layer="91"/>
-<pinref part="RX_CLK0" gate="G$1" pin="P$1"/>
 <wire x1="81.28" y1="5.08" x2="81.28" y2="12.7" width="0.1524" layer="91"/>
 <junction x="81.28" y="12.7"/>
 <label x="86.36" y="-2.54" size="1.778" layer="95" rot="R90"/>
-</segment>
-</net>
+<pinref part="QSD_CLK0" gate="G$1" pin="PIN0"/>
+<wire x1="81.74" y1="-7.7" x2="81.28" y2="-7.7" width="0.1524" layer="91"/>
+<wire x1="81.28" y1="-7.7" x2="81.28" y2="5.08" width="0.1524" layer="91"/>
+</segment>
+</net>
