File: projects/RADIO/SDR_reciever_board_v2.0_mini_try02/sdr_3157.brd (EAGLE design)
At the start: 60 x 75 mm, 53 parts, among them IC1 LM1117-33, U1 NE5532D, U4 SN74LVC1G3157DBVR, U6 SN74LVC1G3157DBVR

Commit message: Update
Parts:
- moved C8 0.71 mm to (15.0, 39.0)
Routing:
- net N$8: track 6.96 -> 5.83 mm
Changed lines of the file:
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@@
 <attribute name="VALUE" x="34.103" y="15.484" locked="yes" size="1.27" layer="27" rot="R180"/>
 </element>
-<element name="C8" library="mylib" package="C0805" value="1uF" x="15.5" y="38.5" locked="yes" smashed="yes" rot="R90">
-<attribute name="NAME" x="13.595" y="38.5" locked="yes" size="1.27" layer="25" rot="R90"/>
-<attribute name="VALUE" x="18.04" y="37.23" locked="yes" size="1.27" layer="27" rot="R90"/>
+<element name="C8" library="mylib" package="C0805" value="1uF" x="15" y="39" smashed="yes" rot="R90">
+<attribute name="NAME" x="13.095" y="39" size="1.27" layer="25" rot="R90"/>
+<attribute name="VALUE" x="17.54" y="37.73" size="1.27" layer="27" rot="R90"/>
 </element>
 <element name="C9" library="rcl" package="C0805" package3d_urn="urn:adsk.eagle:package:23617/2" value="1uF" x="23.5" y="39" locked="yes" smashed="yes" rot="R90">
@@
 <via x="54" y="44" extent="1-16" drill="1" diameter="2" shape="octagon"/>
 <wire x1="46" y1="44" x2="54" y2="44" width="0.6096" layer="16"/>
-<wire x1="25.4" y1="50.595" x2="28.5" y2="40.25" width="0" layer="19" extent="1-1"/>
 </signal>
 <signal name="N$3">
@@
 <contactref element="C8" pad="1"/>
 <contactref element="C15" pad="1"/>
-<wire x1="14.1" y1="37.55" x2="13" y2="36.45" width="0.8128" layer="1"/>
-<wire x1="13" y1="36.45" x2="13" y2="35.45" width="0.8128" layer="1"/>
-<wire x1="15.5" y1="37.55" x2="14.1" y2="37.55" width="0.8128" layer="1"/>
 <wire x1="10" y1="35.45" x2="13" y2="35.45" width="1.016" layer="1"/>
-<wire x1="15.5" y1="37.55" x2="15.5" y2="37.25" width="0" layer="19" extent="1-1"/>
+<wire x1="13" y1="35.7525" x2="14.9975" y2="37.75" width="1.016" layer="1"/>
+<wire x1="14.9975" y1="37.75" x2="15" y2="37.75" width="1.016" layer="1"/>
+<wire x1="13" y1="35.45" x2="13" y2="35.7525" width="0" layer="19" extent="1-1"/>
 <wire x1="10" y1="35.75" x2="10" y2="35.45" width="0" layer="19" extent="1-1"/>
-<wire x1="13" y1="35.7525" x2="15.5" y2="37.25" width="0" layer="19" extent="1-1"/>
 </signal>
 <signal name="N$9">
@@
 <contactref element="R8" pad="1"/>
 <wire x1="18" y1="40.55" x2="18" y2="40.5" width="0.8128" layer="1"/>
-<wire x1="18" y1="40.5" x2="16.95" y2="39.45" width="0.8128" layer="1"/>
-<wire x1="15.5" y1="39.45" x2="16.95" y2="39.45" width="0.8128" layer="1"/>
-<wire x1="18" y1="40.55" x2="18" y2="40.2475" width="0" layer="19" extent="1-1"/>
-<wire x1="15.5" y1="39.75" x2="15.5" y2="39.45" width="0" layer="19" extent="1-1"/>
+<wire x1="18" y1="40.5" x2="17.95" y2="40.45" width="0.8128" layer="1"/>
+<wire x1="15" y1="40.25" x2="17.75" y2="40.25" width="1.016" layer="1"/>
+<wire x1="17.75" y1="40.25" x2="18" y2="40.5" width="1.016" layer="1"/>
+<wire x1="17.95" y1="40.45" x2="18" y2="40.2475" width="0" layer="19" extent="1-1"/>
 </signal>
 <signal name="N$13">

Commit message: update lib
Parts:
- removed R1: 7k5, mylib:C0805
- removed TM2: 5k, rcl:RTRIM3296W
- added P_1: SMD_PIN, mylib:SMD_PIN
- added R3: 10k, mylib:R0805W
- C9: device rcl:C0805 -> mylib:C0805
- COS, RF_IN, RF_IN1, SIN: value (none) -> 2X_SMD_PTH_PIN; device mylib:2XSMD_PIN -> mylib:2X_SMD_PTH
- moved COS 7.10 mm to (17.2, 10.5)
- moved SIN 6.58 mm to (43.0, 11.0), turned to 90 degrees
- moved RF_IN1 6.40 mm to (51.5, 47.0), turned to 180 degrees
- moved C27 6.04 mm to (33.0, 11.0)
- moved R23 5.85 mm to (37.0, 11.0)
- moved R19 5.39 mm to (38.0, 31.0)
- moved C16 5.02 mm to (38.0, 36.5), turned to 270 degrees
- moved C12 4.74 mm to (41.5, 36.5)
- moved C2 4.47 mm to (21.0, 59.0)
- moved Q 4.27 mm to (20.2, 64.0)
- moved C5 3.50 mm to (8.00, 49.5), turned to 270 degrees
- moved R18 3.50 mm to (31.5, 31.0)
- moved R6 3.35 mm to (8.00, 44.5)
- moved R24 3.35 mm to (37.0, 18.3), turned to 270 degrees
- moved U6 3.20 mm to (34.5, 24.5)
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Connections:
- removed net N$41: R1.2, TM2.3
- net 12V: now also P_1.P$1, RF_IN1.T$2
- net COS_IN: now also COS.T$2
- net GND: now also COS.T$1, RF_IN.T$1, RF_IN1.T$1, SIN.T$1
- net N$1: now also RF_IN.T$2
- net N$19: now also R3.1; no longer R1.1
- net N$24: now also R3.2; no longer TM2.1, TM2.2
- net SIN_IN: now also SIN.T$2
Routing:
- net GND: track 71.9 -> 59.4 mm, vias 8 -> 6
- net 12V: track 101.1 -> 108.7 mm
- net N$24: track 28.7 -> 22.2 mm
- net SIN_IN: track 11.4 -> 16.2 mm
- net COS_IN: track 9.77 -> 13.7 mm
- net ANTENNA: track 33.6 -> 29.8 mm
- net N$20: track 26.9 -> 29.9 mm
- net N$25: track 10.1 -> 13.0 mm
- net N$5: track 8.27 -> 5.43 mm
- net N$14: track 2.60 -> 5.19 mm
- net N$41: track 2.57 -> 0.00 mm
- net N$7: track 8.32 -> 5.81 mm
- net VCC: track 63.0 -> 60.6 mm
- net N$17: track 19.1 -> 16.9 mm
- net N$21: track 21.8 -> 23.9 mm
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
Commit message: Update
Parts:
- added 3V3: 2X_SMD_PTH_PIN, mylib:2X_SMD_PTH
- added H5, H6: MOUNT-PAD-ROUND3.0, holes:3,0-PAD
- C11, C12, C8, C9: device mylib:C0805 -> mylib:C0805K
- C3, C4: device rcl:C050-045X075 -> mylib:C0805K
- I, Q: value (none) -> 2X_SMD_PTH_PIN; device mylib:2XSMD_PIN -> mylib:2X_SMD_PTH
- P_1: value SMD_PIN -> SMD_PTH_PIN; device mylib:SMD_PIN -> mylib:SMD_PTH_PIN
- moved C14 43.1 mm to (7.00, 22.0), turned to 270 degrees
- moved C13 41.2 mm to (10.5, 21.8), turned to 270 degrees
- moved C10 6.60 mm to (28.5, 29.7), turned to 270 degrees
- moved TM1 3.61 mm to (13.0, 55.5)
- moved RF_IN1 3.50 mm to (51.5, 43.5)
- moved R10 2.55 mm to (41.7, 44.9)
- moved R7 2.26 mm to (12.8, 45.0)
- moved R3 2.14 mm to (42.1, 52.4)
- moved C9 2.12 mm to (25.0, 37.0)
- moved IC1 2.12 mm to (50.5, 32.5)
- moved P_1 1.98 mm to (6.50, 37.2)
- moved C1 1.80 mm to (32.5, 60.5)
- moved C2 1.50 mm to (21.0, 60.5)
- moved C21 1.50 mm to (23.5, 29.7)
- moved C5 1.50 mm to (8.00, 51.0)
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- renumbered U4 to U2, U6 to U3
Connections:
- net 12V: now also P_1.P$2
- net GND: now also 3V3.P$1, 3V3.T$1, H5.B3,0, H6.B3,0, I.T$1, Q.T$2
- net N$10: now also C11.P$1
- net N$11: now also C12.P$1
- net N$12: now also C8.P$2
- net N$13: now also C9.P$2
- net N$14: now also C11.P$2
- net N$15: now also C12.P$2
- net N$17: now also C3.P$1
- net N$19: now also C4.P$1
- net N$21: now also C3.P$2
- net N$22: now also Q.T$1
- net N$23: now also I.T$2
- net N$24: now also C4.P$2
- net N$8: now also C8.P$1
- net N$9: now also C9.P$1
- net VCC: now also 3V3.P$2, 3V3.T$2
Routing:
- net VCC: track 60.6 -> 74.0 mm
- net GND: track 59.4 -> 46.5 mm
- net N$24: track 22.2 -> 26.6 mm
- net SIN_IN: track 16.2 -> 20.5 mm
- net N$11: track 6.37 -> 10.5 mm
- net 12V: track 108.7 -> 104.8 mm
- net N$19: track 17.8 -> 20.8 mm
- net N$10: track 5.67 -> 8.26 mm
- net N$12: track 2.91 -> 5.35 mm
- net N$18: track 12.3 -> 14.7 mm
- net N$8: track 6.13 -> 8.53 mm
- net N$17: track 16.9 -> 19.3 mm
- net N$21: track 23.9 -> 26.0 mm
- net N$20: track 29.9 -> 31.9 mm
- net N$25: track 13.0 -> 14.9 mm
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
Commit message: update
Parts:
- moved C10 8.75 mm to (33.0, 37.2), turned to 90 degrees
- moved C21 7.42 mm to (24.1, 37.1), turned to 270 degrees
- moved R17 6.15 mm to (26.8, 29.9)
- moved R16 5.15 mm to (15.5, 27.0)
- moved U2 3.20 mm to (20.2, 24.5)
- moved C15 2.43 mm to (11.9, 31.0), turned to 180 degrees
- moved C2 1.95 mm to (22.9, 60.5)
- moved C11 1.85 mm to (30.1, 37.1)
- moved Q 1.85 mm to (22.1, 64.4)
- moved R18 1.81 mm to (30.2, 29.9)
- moved C9 1.80 mm to (26.8, 37.0)
- moved R5 1.50 mm to (15.5, 45.0)
- moved R8 1.50 mm to (19.0, 40.8)
- moved C13 1.00 mm to (9.50, 21.8)
- moved C14 1.00 mm to (6.00, 22.0)
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Routing:
- net GND: track 46.5 -> 32.5 mm, vias 6 -> 4
- net ANTENNA: track 30.8 -> 27.6 mm
- net N$3: track 6.52 -> 3.75 mm
- net N$4: track 4.70 -> 7.18 mm
- net VCC: track 74.0 -> 75.5 mm
- net N$14: track 5.26 -> 3.87 mm
- net N$8: track 8.53 -> 9.92 mm
- net N$13: track 5.36 -> 4.02 mm
- net N$9: track 8.20 -> 7.28 mm
- net N$5: track 4.02 -> 4.80 mm
- net COS_IN: track 14.8 -> 15.5 mm
- net N$10: track 8.26 -> 7.56 mm
- net N$18: track 14.7 -> 14.1 mm
- net N$11: track 10.5 -> 11.0 mm

Commit message: update
Parts:
- moved C21 0.35 mm to (23.8, 37.1)
- moved C10 0.20 mm to (33.2, 37.2)
Routing:
- net N$22: track 3.92 -> 7.01 mm
- net GND: track 32.5 -> 29.5 mm
- net N$23: track 3.96 -> 6.96 mm
- net 12V: track 104.9 -> 104.3 mm

Commit message: Update
Parts:
- removed H1, H2, H3, H4: MOUNT-PAD-ROUND3.0, holes:3,0-PAD
- added IC2: L7805CV, L7805CV:TO255P460X1020X2008-3P
- added L1: DR74, inductors:DR74
- added L2: (no value), mylib:M0805
- moved RF_IN1 20.5 mm to (51.0, 64.0), turned to 90 degrees
- moved C17 11.4 mm to (49.5, 56.0), turned to 180 degrees
- moved C7 11.1 mm to (49.5, 52.0), turned to 0 degrees
- moved H5 9.00 mm to (63.0, 21.0)
- moved H6 9.00 mm to (63.0, 54.0)
- moved IC1 5.70 mm to (54.0, 28.0)
- moved C10 1.50 mm to (31.7, 37.2)
- moved I 1.50 mm to (31.7, 64.4)
- moved 3V3 1.50 mm to (44.5, 22.8)
- moved C1 1.50 mm to (31.0, 60.5)
- moved C11 1.50 mm to (28.6, 37.1)
- moved C13 1.50 mm to (8.00, 21.8)
- moved C14 1.50 mm to (4.50, 22.0)
- moved C15 1.50 mm to (10.4, 31.0)
- moved C2 1.50 mm to (21.4, 60.5)
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Connections:
- new net 5V: IC1.3, IC2.3
- new net VIN: L1.1, L2.1, L2.P$1, RF_IN1.P$2, RF_IN1.T$2
- net 12V: now also IC2.1, L1.2, L2.2, L2.P$2; no longer IC1.3, RF_IN1.P$2, RF_IN1.T$2
- net GND: now also IC2.2; no longer H1.B3,0, H2.B3,0, H3.B3,0, H4.B3,0
Routing:
- net VIN: track 0.00 -> 32.6 mm
- net 5V: track 0.00 -> 10.9 mm
- net 12V: track 104.3 -> 110.6 mm
- net GND: track 29.5 -> 33.8 mm
- net VCC: track 75.9 -> 79.7 mm
- net N$19: track 21.5 -> 19.0 mm
- net N$17: track 19.3 -> 21.7 mm
- net N$24: track 26.6 -> 24.5 mm
- net N$16: track 15.9 -> 17.4 mm
- net N$21: track 25.7 -> 27.2 mm
- net N$18: track 14.6 -> 13.1 mm
- net N$8: track 9.92 -> 10.4 mm
- net N$12: track 5.55 -> 5.05 mm
Other:
- board size 60 x 75 mm -> 70 x 75 mm

Commit message: Update
Parts:
- removed P_1: SMD_PTH_PIN, mylib:SMD_PTH_PIN
- added C18, C19, C20, C22, C23, C24: (no value), mylib:C0805
- added L3: DR74, inductors:DR74
- added L4: (no value), mylib:M0805
- moved C14 45.1 mm to (48.5, 32.0), turned to 90 degrees
- moved C13 44.6 mm to (51.5, 31.7), turned to 90 degrees
- moved L1 16.4 mm to (51.0, 51.5)
- moved IC1 15.0 mm to (60.9, 41.4), turned to 0 degrees
- moved C7 11.4 mm to (40.5, 59.0)
- moved C17 11.1 mm to (40.5, 62.5)
- moved L2 10.8 mm to (56.0, 51.6)
- moved R16 6.25 mm to (7.75, 27.2)
- moved R17 6.08 mm to (19.2, 30.9)
- moved U2 6.02 mm to (12.7, 25.0)
- moved R2 4.10 mm to (11.1, 52.3)
- moved C15 4.03 mm to (6.40, 31.5)
- moved 3V3 4.00 mm to (40.5, 22.7), turned to 0 degrees
- moved R3 3.54 mm to (37.1, 52.9)
- moved Q 3.17 mm to (17.6, 63.2)
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Connections:
- new net N$6: C13.+, C14.1, IC1.2, IC1.4, L3.2, L4.1, L4.P$1
- net 12V: now also C18.1, C19.1, C20.1; no longer P_1.P$1, P_1.P$2
- net GND: now also C18.2, C19.2, C20.2, C22.2, C23.2, C24.2
- net VCC: now also C22.1, C23.1, C24.1, L3.1, L4.2, L4.P$2; no longer C13.+, C14.1, IC1.2, IC1.4
Routing:
- net N$6: track 0.00 -> 44.5 mm
- net VIN: track 32.6 -> 19.4 mm
- net 5V: track 10.9 -> 6.81 mm
- net N$21: track 27.2 -> 23.6 mm
- net ANTENNA: track 27.6 -> 30.9 mm
- net 12V: track 110.6 -> 107.6 mm
- net GND: track 33.8 -> 31.6 mm
- net N$18: track 13.1 -> 14.8 mm
- net N$24: track 24.5 -> 22.9 mm
- net N$20: track 31.8 -> 30.3 mm
- net N$8: track 10.4 -> 11.9 mm
- net COS_IN: track 15.5 -> 14.1 mm
- net VCC: track 79.7 -> 78.3 mm
- net N$28: track 4.02 -> 2.71 mm
- net N$9: track 7.63 -> 8.83 mm
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
Commit message: Update
Parts:
- removed RF_IN1: 2X_SMD_PTH_PIN, mylib:2X_SMD_PTH
- removed R_ATT: 20, rcl:R1210
- added C25, C26, C28, C29: (no value), mylib:C0805
- added CF1: 22nF, mylib:C0805
- added JP1: JUMPER-SMT_3_1-NC_PASTE_NO-SILK, SparkFun-Jumpers:SMT-JUMPER_3_1-NC_PASTE_NO-SILK
- added LF1: 20, mylib:M0805
- added MC_3V3, VIN: 2X_SMD_PTH_PIN, mylib:2X_SMD_PTH
- C6: value 22nF -> (none)
- moved C6 50.6 mm to (51.9, 59.4), turned to 180 degrees
- moved C14 31.2 mm to (52.0, 63.0), turned to 180 degrees
- moved R23 28.5 mm to (5.70, 20.2), turned to 270 degrees
- moved R24 23.0 mm to (9.50, 20.2)
- moved C27 21.5 mm to (7.10, 12.4), turned to 180 degrees
- moved C13 9.00 mm to (60.5, 31.8), turned to 270 degrees
- moved U$3 8.55 mm to (14.7, 16.5), turned to 0 degrees
- moved RF_IN 4.98 mm to (27.1, 9.60)
- moved COS 3.98 mm to (16.8, 9.55)
- moved C15 3.20 mm to (9.60, 31.5), turned to 0 degrees
- moved R4 2.72 mm to (32.1, 46.8)
- moved U2 2.50 mm to (15.2, 25.0)
- moved 3V3 2.09 mm to (38.5, 23.3), turned to 180 degrees
- moved IC2 1.80 mm to (49.9, 42.2)
- moved C17 1.58 mm to (40.0, 64.0)
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Connections:
- removed net N$2: C6.1, R_ATT.1
- new net 3.3V: C22.1, C23.1, C24.1, JP1.1, L3.1, L4.2, L4.P$2, MC_3V3.P$2, MC_3V3.T$2
- net 5V: now also C25.1, C26.1, C28.1, JP1.3
- net ANTENNA: now also CF1.2, LF1.2, LF1.P$2; no longer R_ATT.2
- net GND: now also C25.2, C26.2, C28.2, C29.2, C6.2, CF1.1, MC_3V3.P$1, MC_3V3.T$1, VIN.P$2, VIN.T$2; no longer RF_IN1.P$1, RF_IN1.T$1
- net N$1: now also LF1.1, LF1.P$1; no longer C6.2
- net N$6: no longer C14.1
- net VCC: now also JP1.2; no longer C22.1, C23.1, C24.1, L3.1, L4.2, L4.P$2
- net VIN: now also C14.1, C29.1, C6.1, VIN.P$1, VIN.T$1; no longer RF_IN1.P$2, RF_IN1.T$2
Routing:
- net 3.3V: track 0.00 -> 35.8 mm
- net VCC: track 78.3 -> 48.8 mm
- net 5V: track 6.81 -> 32.3 mm
- net VIN: track 19.4 -> 29.8 mm
- net N$1: track 5.72 -> 16.0 mm
- net N$6: track 44.5 -> 35.3 mm
- net N$18: track 14.8 -> 10.8 mm
- net 12V: track 107.6 -> 111.2 mm
- net N$2: track 3.42 -> 0.00 mm
- net N$4: track 7.69 -> 5.36 mm
- net N$25: track 14.9 -> 12.8 mm
- net N$3: track 4.25 -> 6.25 mm
- net GND: track 31.6 -> 29.6 mm
- net N$7: track 6.02 -> 4.29 mm
- net N$21: track 23.6 -> 25.3 mm
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