File: projects/RADIO/SDR_reciever_board_v2.0_mini_try02/sdr_3157.brd (EAGLE design)
At the start: 70 x 75 mm, 69 parts, among them IC1 LM1117-33, IC2 L7805CV, U1 NE5532D, U2 SN74LVC1G3157DBVR, U3 SN74LVC1G3157DBVR

Commit message: Upload
Parts:
- moved H5 1.00 mm to (62.0, 21.0)
- moved H6 1.00 mm to (62.0, 54.0)
Other:
- board size 70 x 75 mm -> 68 x 75 mm
Changed lines of the file:
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@@
 <board>
 <plain>
-<wire x1="0" y1="0" x2="70" y2="0" width="0.5" layer="20"/>
-<wire x1="70" y1="0" x2="70" y2="75" width="0.5" layer="20"/>
-<wire x1="70" y1="75" x2="0" y2="75" width="0.5" layer="20"/>
+<wire x1="0" y1="0" x2="68" y2="0" width="0.5" layer="20"/>
+<wire x1="68" y1="0" x2="68" y2="75" width="0.5" layer="20"/>
+<wire x1="68" y1="75" x2="0" y2="75" width="0.5" layer="20"/>
 <wire x1="0" y1="75" x2="0" y2="0" width="0.5" layer="20" locked="yes"/>
 <wire x1="17.5" y1="1.5" x2="54" y2="1.5" width="1.5" layer="41" style="shortdash"/>
@@
 <wire x1="7.5" y1="50" x2="7.5" y2="51" width="1.016" layer="41"/>
 <wire x1="26.5" y1="61" x2="26.5" y2="59" width="1.016" layer="41"/>
-<dimension x1="0" y1="0" x2="70" y2="0" x3="35" y3="-12.5" textsize="1.778" layer="47"/>
 <dimension x1="0" y1="75" x2="0" y2="0" x3="-5" y3="37.5" textsize="1.778" layer="47"/>
 <dimension x1="63" y1="21" x2="63" y2="54" x3="77.5" y3="37.5" textsize="1.778" layer="47"/>
 <dimension x1="16.75" y1="9.55" x2="37.75" y2="9.45" x3="27.183409375" y3="-4.48420625" textsize="1.778" layer="47"/>
 <wire x1="15" y1="16.5" x2="12" y2="16.5" width="1.016" layer="41"/>
+<dimension x1="0" y1="0" x2="68" y2="0" x3="34" y3="-10.5" textsize="1.778" layer="47"/>
 </plain>
 <attributes>
@@
 <attribute name="VALUE" x="37.735" y="51.64" size="1.27" layer="27" rot="R180"/>
 </element>
-<element name="H5" library="holes" library_urn="urn:adsk.eagle:library:237" package="3,0-PAD" package3d_urn="urn:adsk.eagle:package:14280/1" value="MOUNT-PAD-ROUND3.0" x="63" y="21" locked="yes" smashed="yes">
-<attribute name="POPULARITY" value="17" x="63" y="21" locked="yes" size="1.778" layer="27" display="off"/>
-</element>
-<element name="H6" library="holes" library_urn="urn:adsk.eagle:library:237" package="3,0-PAD" package3d_urn="urn:adsk.eagle:package:14280/1" value="MOUNT-PAD-ROUND3.0" x="63" y="54" locked="yes" smashed="yes">
-<attribute name="POPULARITY" value="17" x="63" y="54" locked="yes" size="1.778" layer="27" display="off"/>
+<element name="H5" library="holes" library_urn="urn:adsk.eagle:library:237" package="3,0-PAD" package3d_urn="urn:adsk.eagle:package:14280/1" value="MOUNT-PAD-ROUND3.0" x="62" y="21" locked="yes" smashed="yes">
+<attribute name="POPULARITY" value="17" x="62" y="21" locked="yes" size="1.778" layer="27" display="off"/>
+</element>
+<element name="H6" library="holes" library_urn="urn:adsk.eagle:library:237" package="3,0-PAD" package3d_urn="urn:adsk.eagle:package:14280/1" value="MOUNT-PAD-ROUND3.0" x="62" y="54" locked="yes" smashed="yes">
+<attribute name="POPULARITY" value="17" x="62" y="54" locked="yes" size="1.778" layer="27" display="off"/>
 </element>
 <element name="3V3" library="mylib" package="2X_SMD_PTH" value="2X_SMD_PTH_PIN" x="38.5" y="23.3" smashed="yes" rot="R180"/>

Commit message: update
Parts:
- added C30: (no value), mylib:E5-5
- added H1: MOUNT-PAD-ROUND3.0, holes:3,0-PAD
- CF1: value 22nF -> 150pF; device mylib:C0805 -> mylib:C0805K
- LF1: value 20 -> 390nH
- moved R23 7.85 mm to (6.95, 12.4), turned to 180 degrees
- moved C16 7.00 mm to (36.6, 30.9), turned to 0 degrees
- moved C10 6.70 mm to (28.6, 31.0), turned to 0 degrees
- moved IC2 5.41 mm to (45.4, 39.2)
- moved C28 4.65 mm to (48.5, 28.1)
- moved C25 4.61 mm to (41.9, 28.2)
- moved C26 4.61 mm to (45.2, 28.1)
- moved IC1 4.61 mm to (56.9, 36.9)
- moved R19 4.48 mm to (36.8, 27.0), turned to 0 degrees
- moved C27 4.00 mm to (7.10, 8.45)
- moved L4 3.68 mm to (52.9, 19.1)
- moved JP1 3.66 mm to (42.0, 22.3)
- moved L3 3.20 mm to (48.0, 19.0)
- moved C8 3.16 mm to (9.60, 36.6)
- moved U1 3.16 mm to (22.0, 52.0)
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Connections:
- net 12V: now also C30.+
- net ANTENNA: now also CF1.P$2
- net GND: now also C30.-, CF1.P$1, H1.B3,0
Routing:
- net GND: track 29.6 -> 36.5 mm
- net N$18: track 10.8 -> 15.4 mm
- net N$21: track 25.3 -> 21.6 mm
- net 3.3V: track 35.8 -> 33.0 mm
- net N$17: track 21.4 -> 18.7 mm
- net VCC: track 48.8 -> 46.1 mm
- net N$6: track 35.3 -> 33.0 mm
- net N$14: track 3.87 -> 6.01 mm
- net N$19: track 18.5 -> 20.6 mm
- net N$13: track 4.02 -> 6.04 mm
- net N$11: track 10.4 -> 8.42 mm
- net N$8: track 12.0 -> 10.2 mm
- net N$24: track 24.2 -> 22.5 mm
- net ANTENNA: track 30.5 -> 32.2 mm
- net N$12: track 4.74 -> 6.39 mm
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Other:
- board size 68 x 75 mm -> 65 x 75 mm
