File: projects/RADIO/SDR_reciever_board_v2.0_mini_try02/sdr_3157.sch (EAGLE design)
At the start: 53 parts, among them IC1 LM1117-33, U1 NE5532D, U4 SN74LVC1G3157DBVR, U6 SN74LVC1G3157DBVR

Commit message: update lib
Parts:
- removed R1: 7k5, mylib:C_0805_SMD
- removed TM2: 5k, rcl:R-TRIMM3296W
- added P_1: SMD_PIN, mylib:SMD_PIN
- added R3: 10k, mylib:R_0805_SMD
- C9: device rcl:C-EUC0805 -> mylib:C_0805_SMD
- COS, RF_IN, RF_IN1, SIN: value (none) -> 2X_SMD_PTH_PIN; device mylib:2X_SMD_PIN -> mylib:2X_SMD_PTH_PIN
Connections:
- removed net N$41: R1.2, TM2.E
- net 12V: now also P_1.P$1
- net N$19: now also R3.1; no longer R1.1
- net N$24: now also R3.2; no longer TM2.A, TM2.S
Changed lines of the file:
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@@
 <part name="R19" library="mylib" deviceset="R_0805_SMD" device="" value="20"/>
 <part name="C8" library="mylib" deviceset="C_0805_SMD" device="" value="1uF"/>
-<part name="C9" library="rcl" deviceset="C-EU" device="C0805" package3d_urn="urn:adsk.eagle:package:23617/2" value="1uF"/>
+<part name="C9" library="mylib" deviceset="C_0805_SMD" device="" value="1uF"/>
 <part name="C11" library="mylib" deviceset="C_0805_SMD" device="" value="1uF"/>
 <part name="C12" library="mylib" deviceset="C_0805_SMD" device="" value="1uF"/>
@@
 <part name="GND8" library="supply1" library_urn="urn:adsk.eagle:library:371" deviceset="GND" device=""/>
 <part name="R2" library="mylib" deviceset="R_0805_SMD" device="" value="7k5"/>
-<part name="R1" library="mylib" deviceset="C_0805_SMD" device="" value="7k5"/>
 <part name="C2" library="rcl" deviceset="C-EU" device="050-045X075" package3d_urn="urn:adsk.eagle:package:23638/1" value="1uF"/>
 <part name="C1" library="rcl" deviceset="C-EU" device="050-045X075" package3d_urn="urn:adsk.eagle:package:23638/1" value="1uF"/>
@@
 <part name="GND4" library="supply1" library_urn="urn:adsk.eagle:library:371" deviceset="GND" device=""/>
 <part name="SUPPLY9" library="SparkFun-PowerSymbols" deviceset="12V" device=""/>
-<part name="TM2" library="rcl" deviceset="R-TRIMM" device="3296W" package3d_urn="urn:adsk.eagle:package:26033/1" value="5k"/>
 <part name="C6" library="mylib" deviceset="C_0805_SMD" device="" value="22nF"/>
 <part name="GND14" library="supply1" library_urn="urn:adsk.eagle:library:371" deviceset="GND" device=""/>
@@
 <part name="GND20" library="supply1" library_urn="urn:adsk.eagle:library:371" deviceset="GND" device=""/>
 <part name="GND23" library="supply1" library_urn="urn:adsk.eagle:library:371" deviceset="GND" device=""/>
-<part name="RF_IN" library="mylib" deviceset="2X_SMD_PIN" device=""/>
-<part name="COS" library="mylib" deviceset="2X_SMD_PIN" device=""/>
-<part name="SIN" library="mylib" deviceset="2X_SMD_PIN" device=""/>
+<part name="RF_IN" library="mylib" deviceset="2X_SMD_PTH_PIN" device=""/>
+<part name="COS" library="mylib" deviceset="2X_SMD_PTH_PIN" device=""/>
+<part name="SIN" library="mylib" deviceset="2X_SMD_PTH_PIN" device=""/>
 <part name="I" library="mylib" deviceset="2X_SMD_PIN" device=""/>
 <part name="Q" library="mylib" deviceset="2X_SMD_PIN" device=""/>
@@
 <part name="GND25" library="supply1" library_urn="urn:adsk.eagle:library:371" deviceset="GND" device=""/>
 <part name="GND26" library="supply1" library_urn="urn:adsk.eagle:library:371" deviceset="GND" device=""/>
-<part name="RF_IN1" library="mylib" deviceset="2X_SMD_PIN" device=""/>
+<part name="RF_IN1" library="mylib" deviceset="2X_SMD_PTH_PIN" device=""/>
+<part name="P_1" library="mylib" deviceset="SMD_PIN" device=""/>
+<part name="R3" library="mylib" deviceset="R_0805_SMD" device="" value="10k"/>
 </parts>
 <sheets>
@@
 <attribute name="VALUE" x="138.43" y="88.138" size="1.778" layer="96"/>
 </instance>
-<instance part="R1" gate="G$1" x="147.32" y="40.64" smashed="yes">
-<attribute name="NAME" x="146.05" y="42.1386" size="1.778" layer="95"/>
-<attribute name="VALUE" x="143.51" y="37.338" size="1.778" layer="96"/>
-</instance>
 <instance part="C2" gate="G$1" x="172.72" y="66.04" smashed="yes">
 <attribute name="NAME" x="176.784" y="63.881" size="1.778" layer="95"/>
@@
 <attribute name="VALUE" x="155.194" y="-17.78" size="1.778" layer="96" rot="R270" align="bottom-center"/>
 </instance>
-<instance part="TM2" gate="G$1" x="160.02" y="40.64" smashed="yes" rot="R90">
-<attribute name="NAME" x="161.29" y="47.371" size="1.778" layer="95" rot="R180"/>
-</instance>
 <instance part="C6" gate="G$1" x="-10.16" y="63.5" smashed="yes" rot="R270">
 <attribute name="NAME" x="-12.319" y="59.436" size="1.778" layer="95" rot="R270"/>
@@
 <instance part="RF_IN1" gate="G$1" x="88.9" y="160.02" smashed="yes">
 <attribute name="NAME" x="89.98" y="166.12" size="1.27" layer="95"/>
+</instance>
+<instance part="P_1" gate="G$1" x="76.2" y="154.94" smashed="yes" rot="R270"/>
+<instance part="R3" gate="G$1" x="152.4" y="40.64" smashed="yes">
+<attribute name="NAME" x="151.13" y="42.1386" size="1.778" layer="95"/>
+<attribute name="VALUE" x="148.59" y="37.338" size="1.778" layer="96"/>
 </instance>
 </instances>
@@
 <segment>
 <pinref part="U1" gate="B" pin="-IN"/>
-<pinref part="R1" gate="G$1" pin="1"/>
 <wire x1="137.16" y1="25.4" x2="139.7" y2="25.4" width="0.1524" layer="91"/>
 <wire x1="137.16" y1="25.4" x2="137.16" y2="27.94" width="0.1524" layer="91"/>
 <wire x1="137.16" y1="27.94" x2="137.16" y2="33.02" width="0.1524" layer="91"/>
 <wire x1="137.16" y1="33.02" x2="137.16" y2="40.64" width="0.1524" layer="91"/>
-<wire x1="137.16" y1="40.64" x2="147.32" y2="43.18" width="0.1524" layer="91"/>
 <pinref part="C4" gate="G$1" pin="1"/>
 <wire x1="142.24" y1="33.02" x2="137.16" y2="33.02" width="0.1524" layer="91"/>
@@
 <wire x1="114.3" y1="27.94" x2="137.16" y2="27.94" width="0.1524" layer="91"/>
 <junction x="137.16" y="27.94"/>
+<pinref part="R3" gate="G$1" pin="1"/>
+<wire x1="147.32" y1="40.64" x2="137.16" y2="40.64" width="0.1524" layer="91"/>
 </segment>
 </net>
@@
 <wire x1="172.72" y1="38.1" x2="172.72" y2="22.86" width="0.1524" layer="91"/>
 <wire x1="172.72" y1="22.86" x2="167.64" y2="22.86" width="0.1524" layer="91"/>
-<pinref part="TM2" gate="G$1" pin="A"/>
 <wire x1="167.64" y1="22.86" x2="154.94" y2="22.86" width="0.1524" layer="91"/>
-<wire x1="165.1" y1="40.64" x2="167.64" y2="40.64" width="0.1524" layer="91"/>
-<wire x1="167.64" y1="40.64" x2="167.64" y2="33.02" width="0.1524" layer="91"/>
 <junction x="167.64" y="22.86"/>
 <pinref part="C4" gate="G$1" pin="2"/>
 <wire x1="167.64" y1="33.02" x2="167.64" y2="22.86" width="0.1524" layer="91"/>
 <wire x1="149.86" y1="33.02" x2="167.64" y2="33.02" width="0.1524" layer="91"/>
+<pinref part="R3" gate="G$1" pin="2"/>
+<wire x1="157.48" y1="40.64" x2="167.64" y2="40.64" width="0.1524" layer="91"/>
+<wire x1="167.64" y1="40.64" x2="167.64" y2="33.02" width="0.1524" layer="91"/>
 <junction x="167.64" y="33.02"/>
-<pinref part="TM2" gate="G$1" pin="S"/>
-<wire x1="160.02" y1="45.72" x2="167.64" y2="45.72" width="0.1524" layer="91"/>
-<wire x1="167.64" y1="45.72" x2="167.64" y2="40.64" width="0.1524" layer="91"/>
-<junction x="167.64" y="40.64"/>
 </segment>
 </net>
@@
 </segment>
 <segment>
-<wire x1="86.44" y1="160.02" x2="66.04" y2="160.02" width="0.1524" layer="91"/>
+<wire x1="86.44" y1="160.02" x2="76.2" y2="160.02" width="0.1524" layer="91"/>
 <pinref part="SUPPLY4" gate="G$1" pin="12V"/>
 <pinref part="RF_IN1" gate="G$1" pin="PIN1"/>
+<pinref part="P_1" gate="G$1" pin="P$1"/>
+<wire x1="76.2" y1="160.02" x2="66.04" y2="160.02" width="0.1524" layer="91"/>
+<wire x1="76.2" y1="154.94" x2="76.2" y2="160.02" width="0.1524" layer="91"/>
+<junction x="76.2" y="160.02"/>
 </segment>
 <segment>
@@
 </segment>
 </net>
-<net name="N$41" class="0">
-<segment>
-<pinref part="R1" gate="G$1" pin="2"/>
-<pinref part="TM2" gate="G$1" pin="E"/>
-<wire x1="154.94" y1="40.64" x2="147.32" y2="35.56" width="0.1524" layer="91"/>
-</segment>
-</net>

Commit message: Update
Parts:
- added 3V3: 2X_SMD_PTH_PIN, mylib:2X_SMD_PTH_PIN
- added H5, H6: MOUNT-PAD-ROUND3.0, holes:MOUNT-PAD-ROUND3.0
- C11, C12, C8, C9: device mylib:C_0805_SMD -> mylib:C_0805_PTH
- C3, C4: device rcl:C-EU050-045X075 -> mylib:C_0805_PTH
- I, Q: value (none) -> 2X_SMD_PTH_PIN; device mylib:2X_SMD_PIN -> mylib:2X_SMD_PTH_PIN
- P_1: value SMD_PIN -> SMD_PTH_PIN; device mylib:SMD_PIN -> mylib:SMD_PTH_PIN
- renumbered U4 to U2, U6 to U3
Connections:
- net GND: now also 3V3.PIN0, H5.MOUNT, H6.MOUNT
- net VCC: now also 3V3.PIN1
Other:
- moved on the sheet: Q, R8, R9

Commit message: Update
Parts:
- removed H1, H2, H3, H4: MOUNT-PAD-ROUND3.0, holes:MOUNT-PAD-ROUND3.0
- added IC2: L7805CV, L7805CV:L7805CV
- added L1: DR74, inductors:DR74
- added L2: (no value), mylib:L_0805_PTH
Connections:
- new net 5V: IC1.INPUT, IC2.OUTPUT
- new net VIN: L1.1, L2.1, RF_IN1.PIN1
- net 12V: now also IC2.INPUT, L1.2, L2.2; no longer IC1.INPUT, RF_IN1.PIN1
- net GND: now also IC2.GROUND; no longer H1.MOUNT, H2.MOUNT, H3.MOUNT, H4.MOUNT
Other:
- moved on the sheet: C17, C7

Commit message: Update
Parts:
- removed P_1: SMD_PTH_PIN, mylib:SMD_PTH_PIN
- added C18, C19, C20, C22, C23, C24: (no value), mylib:C_0805_SMD
- added L3: DR74, inductors:DR74
- added L4: (no value), mylib:L_0805_PTH
Connections:
- new net N$6: C13.+, C14.1, IC1.OUTPUT_1, IC1.OUTPUT_2, L3.2, L4.1
- net 12V: now also C18.1, C19.1, C20.1; no longer P_1.P$1
- net GND: now also C18.2, C19.2, C20.2, C22.2, C23.2, C24.2
- net VCC: now also C22.1, C23.1, C24.1, L3.1, L4.2; no longer C13.+, C14.1, IC1.OUTPUT_1, IC1.OUTPUT_2
Other:
- moved on the sheet: 3V3

Commit message: Update
Parts:
- removed RF_IN1: 2X_SMD_PTH_PIN, mylib:2X_SMD_PTH_PIN
- removed R_ATT: 20, rcl:R-EU_R1210
- added C25, C26, C28, C29: (no value), mylib:C_0805_SMD
- added CF1: 22nF, mylib:C_0805_SMD
- added JP1: JUMPER-SMT_3_1-NC_PASTE_NO-SILK, SparkFun-Jumpers:JUMPER-SMT_3_1-NC_PASTE_NO-SILK
- added LF1: 20, mylib:L_0805_PTH
- added MC_3V3, VIN: 2X_SMD_PTH_PIN, mylib:2X_SMD_PTH_PIN
- C6: value 22nF -> (none)
Connections:
- removed net N$2: C6.1, R_ATT.1
- new net 3.3V: C22.1, C23.1, C24.1, JP1.1, L3.1, L4.2, MC_3V3.PIN1
- net 5V: now also C25.1, C26.1, C28.1, JP1.3
- net ANTENNA: now also CF1.2, LF1.2; no longer R_ATT.2
- net GND: now also C25.2, C26.2, C28.2, C29.2, C6.2, CF1.1, MC_3V3.PIN0, VIN.PIN1; no longer RF_IN1.PIN0
- net N$1: now also LF1.1; no longer C6.2
- net N$6: no longer C14.1
- net VCC: now also JP1.2; no longer C22.1, C23.1, C24.1, L3.1, L4.2
- net VIN: now also C14.1, C29.1, C6.1, VIN.PIN0; no longer RF_IN1.PIN1
Other:
- moved on the sheet: 3V3, C14, C22, C23, C24, C6, U1P

Commit message: update
Parts:
- added C30: (no value), mylib:C_POL
- added H1: MOUNT-PAD-ROUND3.0, holes:MOUNT-PAD-ROUND3.0
- CF1: value 22nF -> 150pF; device mylib:C_0805_SMD -> mylib:C_0805_PTH
- LF1: value 20 -> 390nH
Connections:
- net 12V: now also C30.+
- net GND: now also C30.-, H1.MOUNT
Changed lines of the file:
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@@
 <part name="GND14" library="supply1" library_urn="urn:adsk.eagle:library:371" deviceset="GND" device=""/>
 <part name="SUPPLY3" library="SparkFun-PowerSymbols" deviceset="12V" device=""/>
-<part name="LF1" library="mylib" deviceset="L_0805_PTH" device="" value="20"/>
+<part name="LF1" library="mylib" deviceset="L_0805_PTH" device="" value="390nH"/>
 <part name="GND17" library="supply1" library_urn="urn:adsk.eagle:library:371" deviceset="GND" device=""/>
 <part name="GND13" library="supply1" library_urn="urn:adsk.eagle:library:371" deviceset="GND" device=""/>
@@
 <part name="GND26" library="supply1" library_urn="urn:adsk.eagle:library:371" deviceset="GND" device=""/>
 <part name="SUPPLY21" library="SparkFun-PowerSymbols" deviceset="3.3V" device=""/>
-<part name="CF1" library="mylib" deviceset="C_0805_SMD" device="" value="22nF"/>
+<part name="CF1" library="mylib" deviceset="C_0805_PTH" device="" value="150pF"/>
 <part name="GND36" library="supply1" library_urn="urn:adsk.eagle:library:371" deviceset="GND" device=""/>
 <part name="C6" library="mylib" deviceset="C_0805_SMD" device=""/>
@@
 <part name="SUPPLY23" library="SparkFun-PowerSymbols" deviceset="VIN" device=""/>
 <part name="SUPPLY24" library="SparkFun-PowerSymbols" deviceset="VIN" device=""/>
+<part name="C30" library="mylib" deviceset="C_POL" device=""/>
+<part name="GND40" library="supply1" library_urn="urn:adsk.eagle:library:371" deviceset="GND" device=""/>
+<part name="H1" library="holes" library_urn="urn:adsk.eagle:library:237" deviceset="MOUNT-PAD-ROUND" device="3.0" package3d_urn="urn:adsk.eagle:package:14280/1"/>
+<part name="GND41" library="supply1" library_urn="urn:adsk.eagle:library:371" deviceset="GND" device=""/>
 </parts>
 <sheets>
@@
 <attribute name="VALUE" x="208.026" y="-50.8" size="1.778" layer="96" rot="R90" align="bottom-center"/>
 </instance>
-<instance part="CF1" gate="G$1" x="2.54" y="53.34" smashed="yes" rot="R180">
-<attribute name="NAME" x="-1.524" y="55.499" size="1.778" layer="95" rot="R180"/>
-<attribute name="VALUE" x="1.016" y="58.039" size="1.778" layer="96" rot="R180"/>
+<instance part="CF1" gate="C$1" x="2.54" y="53.34" smashed="yes" rot="R90">
+<attribute name="NAME" x="4.699" y="57.404" size="1.778" layer="95" rot="R90"/>
+<attribute name="VALUE" x="7.239" y="54.864" size="1.778" layer="96" rot="R90"/>
 </instance>
 <instance part="GND36" gate="1" x="2.54" y="43.18" smashed="yes">
@@
 <instance part="SUPPLY24" gate="G$1" x="170.18" y="-149.86" smashed="yes">
 <attribute name="VALUE" x="170.18" y="-147.066" size="1.778" layer="96" align="bottom-center"/>
+</instance>
+<instance part="C30" gate="G$1" x="142.24" y="-104.14" smashed="yes" rot="R180">
+<attribute name="NAME" x="141.097" y="-104.6226" size="1.778" layer="95" rot="R180"/>
+<attribute name="VALUE" x="141.097" y="-99.5426" size="1.778" layer="96" rot="R180"/>
+</instance>
+<instance part="GND40" gate="1" x="142.24" y="-93.98" smashed="yes" rot="R180">
+<attribute name="VALUE" x="144.78" y="-91.44" size="1.778" layer="96" rot="R180"/>
+</instance>
+<instance part="H1" gate="G$1" x="63.5" y="-33.02" smashed="yes">
+<attribute name="NAME" x="66.294" y="-32.4358" size="1.778" layer="95"/>
+</instance>
+<instance part="GND41" gate="1" x="53.34" y="-33.02" smashed="yes" rot="R270">
+<attribute name="VALUE" x="50.8" y="-30.48" size="1.778" layer="96" rot="R270"/>
 </instance>
 </instances>
@@
 </segment>
 <segment>
-<pinref part="CF1" gate="G$1" pin="1"/>
+<pinref part="CF1" gate="C$1" pin="1"/>
 <pinref part="GND36" gate="1" pin="GND"/>
-<wire x1="2.54" y1="45.72" x2="2.54" y2="50.8" width="0.1524" layer="91"/>
+<wire x1="2.54" y1="45.72" x2="2.54" y2="50.038" width="0.1524" layer="91"/>
 </segment>
 <segment>
@@
 <pinref part="VIN" gate="G$1" pin="PIN1"/>
 <wire x1="213.36" y1="-73.66" x2="223.6" y2="-73.66" width="0.1524" layer="91"/>
+</segment>
+<segment>
+<pinref part="C30" gate="G$1" pin="-"/>
+<pinref part="GND40" gate="1" pin="GND"/>
+<wire x1="142.24" y1="-96.52" x2="142.24" y2="-99.06" width="0.1524" layer="91"/>
+</segment>
+<segment>
+<pinref part="H1" gate="G$1" pin="MOUNT"/>
+<pinref part="GND41" gate="1" pin="GND"/>
+<wire x1="55.88" y1="-33.02" x2="60.96" y2="-33.02" width="0.1524" layer="91"/>
 </segment>
 </net>
@@
 <wire x1="-2.54" y1="63.5" x2="2.54" y2="63.5" width="0.1524" layer="91"/>
 <junction x="12.7" y="63.5"/>
-<pinref part="CF1" gate="G$1" pin="2"/>
+<pinref part="CF1" gate="C$1" pin="2"/>
 <wire x1="2.54" y1="63.5" x2="12.7" y2="63.5" width="0.1524" layer="91"/>
-<wire x1="2.54" y1="58.42" x2="2.54" y2="63.5" width="0.1524" layer="91"/>
+<wire x1="2.54" y1="56.642" x2="2.54" y2="63.5" width="0.1524" layer="91"/>
 <junction x="2.54" y="63.5"/>
 </segment>
@@
 <junction x="109.22" y="-116.84"/>
 <pinref part="SUPPLY7" gate="G$1" pin="12V"/>
-<wire x1="134.62" y1="-109.22" x2="134.62" y2="-116.84" width="0.1524" layer="91"/>
+<wire x1="134.62" y1="-109.22" x2="134.62" y2="-111.76" width="0.1524" layer="91"/>
 <junction x="134.62" y="-116.84"/>
-</segment>
-<segment>
+<pinref part="C30" gate="G$1" pin="+"/>
+<wire x1="134.62" y1="-111.76" x2="134.62" y2="-116.84" width="0.1524" layer="91"/>
+<wire x1="134.62" y1="-111.76" x2="142.24" y2="-111.76" width="0.1524" layer="91"/>
+<wire x1="142.24" y1="-111.76" x2="142.24" y2="-106.68" width="0.1524" layer="91"/>
+<junction x="134.62" y="-111.76"/>
+</segment>
+<segment>
