File: projects/RADIO/up_converter/upconverter/upconvertersch.brd (EAGLE design)
At the start: 75 x 50 mm, 20 parts, among them IC1 SA612AN_01,112, IC2 LD1117STR, T1 TRANSFORMER, T2 TRANSFORMER

Commit message: Update
Parts:
- added H1, H2, H3, H4: MOUNT-PAD-ROUND3.0, holes:3,0-PAD
- moved U$1 8.00 mm to (37.5, 7.30)
- moved RF_IN 4.92 mm to (62.8, 12.9)
- moved T2 4.07 mm to (40.1, 19.2)
- moved QG1 2.83 mm to (16.5, 17.0)
- moved C1 2.50 mm to (48.4, 40.8)
- moved C2 2.01 mm to (54.0, 30.0)
- moved C3 2.00 mm to (64.7, 40.6)
- moved C4 2.00 mm to (59.5, 30.0)
- moved C5 2.00 mm to (64.8, 30.0)
- moved L1 2.00 mm to (54.0, 40.7)
- moved L2 2.00 mm to (59.5, 40.7)
- moved R1 2.00 mm to (61.1, 21.4)
- moved T1 2.00 mm to (39.5, 40.8)
- moved 5V 1.00 mm to (12.6, 42.3)
- moved C8 1.00 mm to (13.0, 37.0)
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Connections:
- net GND: now also H1.B3,0, H2.B3,0, H3.B3,0, H4.B3,0
Routing:
- net N$4: track 32.0 -> 24.6 mm
- net N$10: track 14.7 -> 10.2 mm
- net 3.3V: track 40.0 -> 36.3 mm
- net N$2: track 21.3 -> 18.5 mm
- net N$3: track 13.8 -> 11.0 mm
- net VCC: track 27.1 -> 25.1 mm
- net N$1: track 12.8 -> 11.1 mm
- net N$12: track 29.6 -> 28.0 mm
- net N$11: track 8.65 -> 7.26 mm
- net N$13: track 6.29 -> 7.29 mm
- net N$6: track 14.9 -> 15.7 mm
- net N$5: track 8.06 -> 7.56 mm
