File: projects/RADIO/up_converter_2.0/upconverter/upconvertersch.brd (EAGLE design)
At the start: 75 x 50 mm, 20 parts, among them IC1 SA612AN_01,112, IC2 LD1117STR, T1 TRANSFORMER, T2 TRANSFORMER

Commit message: Update
Parts:
- removed U$1: RTL_SDR_CONN, mylib:RTL_SDR_OUT
- added C10: 12pF, mylib:C0805K
- added C11, C12: 15pF, mylib:C0805K
- added C13: 33pF, mylib:C0805K
- added C9: 100pF, mylib:C0805K
- added H1, H2, H3, H4: MOUNT-PAD-ROUND3.0, holes:3,0-PAD
- added L3, L4, L5: 39nH, mylib:M0805
- added RF_OUT: 2X_SMD_PTH_PIN, mylib:2X_SMD_PTH
- QG1: device crystal:DIL14S -> crystal:DIL08S
- moved RF_IN 103.8 mm to (20.1, 102.1), turned to 90 degrees
- moved R1 84.3 mm to (21.8, 94.9), turned to 90 degrees
- moved C5 75.5 mm to (19.2, 88.6), turned to 270 degrees
- moved C4 69.3 mm to (16.2, 82.4), turned to 0 degrees
- moved L2 55.2 mm to (19.2, 76.1), turned to 270 degrees
- moved C3 53.2 mm to (22.2, 69.8), turned to 180 degrees
- moved C2 53.0 mm to (12.7, 60.7), turned to 0 degrees
- moved L1 43.3 mm to (19.2, 63.6)
- moved R2 34.9 mm to (34.0, 5.10), turned to 90 degrees
- moved C1 34.7 mm to (19.2, 54.8), turned to 270 degrees
- moved 5V 34.3 mm to (14.7, 8.10), turned to 180 degrees
- moved QG1 32.5 mm to (51.0, 14.5), turned to 270 degrees
- moved C8 29.6 mm to (20.0, 8.50), turned to 270 degrees
- moved IC2 27.3 mm to (14.8, 17.0), turned to 0 degrees
- moved C6 27.2 mm to (34.2, 10.5), turned to 0 degrees
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Connections:
- new net N$15: C10.1, C10.P$1, C11.1, C11.P$1, C9.2, C9.P$2, L3.2, L3.P$2
- new net N$16: C11.2, C11.P$2, C12.1, C12.P$1, L4.2, L4.P$2
- new net N$17: C12.2, C12.P$2, C13.1, C13.P$1, L5.2, L5.P$2
- new net N$18: C13.2, C13.P$2, RF_OUT.P$2, RF_OUT.T$2
- net 3.3V: now also QG1.8; no longer QG1.14
- net GND: now also C10.2, C10.P$2, H1.B3,0, H2.B3,0, H3.B3,0, H4.B3,0, L3.1, L3.P$1, L4.1, L4.P$1, L5.1, L5.P$1, QG1.4, RF_OUT.P$1, RF_OUT.T$1; no longer QG1.7, U$1.P$2, U$1.P$3
- net N$11: now also QG1.5; no longer QG1.8
- net N$12: now also C9.1, C9.P$1; no longer U$1.P$1
Routing:
- net N$15: track 0.00 -> 20.1 mm
- net N$3: track 13.8 -> 32.2 mm
- net N$12: track 29.3 -> 11.5 mm
- net N$17: track 0.00 -> 13.5 mm
- net N$16: track 0.00 -> 12.8 mm
- net N$18: track 0.00 -> 10.5 mm
- net N$10: track 14.7 -> 8.93 mm
- net N$2: track 21.3 -> 26.4 mm
- net 3.3V: track 40.0 -> 44.5 mm
- net N$11: track 8.65 -> 12.9 mm
- net N$7: track 15.9 -> 11.9 mm
- net N$5: track 8.06 -> 11.6 mm
- net N$8: track 15.2 -> 11.7 mm
- net N$6: track 14.9 -> 11.6 mm
- net N$9: track 9.05 -> 6.29 mm
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Other:
- board size 75 x 50 mm -> 75 x 110 mm
