File: projects/RADIO/TX_SDR/FST3253_TX/tx_board.sch (EAGLE design)
At the start: 24 parts, among them IC2 NE5532N, IC3 NE5532N

Commit message: Update
Parts:
- removed IC3: NE5532N, linear:NE5532N
- added 5VDC, CLK1, CLK2, LINE_OUNT_IN, RF_OUT: 2X_SMD_PTH_PIN, mylib:2X_SMD_PTH_PIN
- added C10, C12, C14, C7: 10uF, mylib:C_0805_SMD
- added C11, C8: 0.022uF, mylib:C_0805_SMD
- added C13: 100nF, mylib:C_0805_SMD
- added C15: 100pF, mylib:C_0805_SMD
- added C16, C17: (no value), mylib:C_0805_SMD
- added C18, C19: (no value), mylib:C_0805_PTH
- added C9: 4.7uF, mylib:C_0805_SMD
- added IC1: NE5532D, linear:NE5532D
- added Q1: 2N3904, transistor-small-signal:2N3904
- added R14, R15: 50k, mylib:R_0805_SMD
- added R16, R17: 10k, mylib:R_0805_SMD
- added R18: 3.3k, mylib:R_0805_SMD
- added R19: 2.2k, mylib:R_0805_SMD
- added R20: 22k, mylib:R_0805_SMD
- added TX_DISABLE: SMD_PTH_PIN, mylib:SMD_PTH_PIN
- C1, C4: value (none) -> 10uF
- C2: value (none) -> 100pF
- C3: value (none) -> 0.022uF
- C5: value 100pF -> 0.022uF
- C6: value 100pF -> 100nF
- IC2: value NE5532N -> NE5532D; device linear:NE5532N -> linear:NE5532D
- R1: value 4.99k -> 10k
- R10, R11, R7, R8: value 10k -> 50k
- R2: value 50k -> 4.99k
- R3: value 50k -> 10k
- R4: value 2.2k -> 10k
- R5: value 3.3k -> 10k
- R6: value 10k -> 2.2k; device mylib:R_0805_SMD -> rcl:R-EU_0204/7
- R9: value 10k -> 2.2k
Connections:
- new net N$18: C19.1, RF_OUT.PIN1
- new net N$19: C1.1, LINE_OUNT_IN.PIN0
- new net N$20: C14.1, LINE_OUNT_IN.PIN1
- new net N$22: C14.2, R12.2
- new net N$23: C1.2, R3.2
- new net N$24: R20.2, TX_DISABLE.P$1
- new net N$25: C12.2, R11.2
- new net N$26: C10.2, R10.2
- new net N$27: C7.2, R8.2
- new net N$29: C13.1, C6.2, C9.2, IC1A.+IN, IC1B.+IN, IC2A.+IN, IC2B.+IN, R6.1, R9.2
- net 0: now also C3.2, R11.1
- net 180: now also C11.2, R7.1
- net 270: now also C8.2, R8.1, U$1.2B3
- net 5V: now also 5VDC.PIN1, IC1P.V+, IC2P.V+, R18.1, R2.2, R6.2; no longer R1.2, R5.1
- net 90: now also C5.2, R10.1
- net CLK0: now also CLK1.PIN0
- net CLK1: now also CLK2.PIN1
- net GND: now also 5VDC.PIN0, C11.1, C13.2, C16.1, C17.1, C18.2, C3.1, C5.1, C6.1, C8.1, C9.1, CLK1.PIN1, CLK2.PIN0, IC1P.V-, IC2P.V-, Q1.E, R19.2, R9.1, RF_OUT.PIN0; no longer C1.1, C2.1, C3.2, R4.2
- net N$1: now also Q1.C, R2.1; no longer R1.1
- net N$10: now also C12.1, C2.2, IC1A.OUT, R1.2, R4.1; no longer C5.2, IC2A.OUT, R12.1, R7.2
- net N$11: now also IC1B.-IN, R1.1, R5.2; no longer IC2B.-IN, R10.2, R7.1
- net N$12: now also C15.1, IC2A.-IN, R12.1; no longer C6.1, IC3A.-IN, R8.1
- net N$13: now also C10.1, C15.2, IC2A.OUT, R17.2; no longer C6.2, IC3A.OUT, R9.2
- net N$14: now also IC2B.-IN, R16.2, R17.1; no longer IC3B.-IN, R11.2, R9.1
- net N$15: now also C4.1, IC1B.OUT, R5.1; no longer IC2B.OUT, R10.1
- net N$16: now also C7.1, IC2B.OUT, R16.1; no longer IC3B.OUT, R11.1
- net N$17: now also C4.2, R7.2; no longer IC3A.+IN, IC3B.+IN
- net N$2: now also R15.2; no longer R2.2
- net N$21: now also Q1.B, R20.1; no longer U$1.2B3
- net N$3: now also R14.2; no longer R3.2
- net N$4: now also R14.1; no longer R3.1
- net N$5: now also R15.1; no longer R2.1
- net N$6: now also C16.2, C17.2, R18.2, R19.1; no longer C1.2, C2.2, R4.1, R5.2
- net N$7: now also C2.1, IC1A.-IN, R3.1, R4.2; no longer C5.1, IC2A.-IN, R12.2, R6.1
- net N$8: now also C18.1; no longer C3.1
- net N$9: now also C19.2; no longer C4.2
Other:
- moved on the sheet: C1, C2, C3, C4, C5, C6, IC2A, IC2B, L1, R1, R10, R11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
