File: projects/RADIO/up_converter_ade_2.0/upconverter/upconvertersch.sch (EAGLE design)
At the start: 32 parts, among them IC1 ADE-1+, IC2 LD1117STR, J1 USB-A-S-S-B-TH

Commit message: update
Parts:
- removed JP1: USB_SOLDER_PADS, SparkFun-Connectors:USB_SOLDER_PADS
- added JH1: (no value), mylib:4X_PIN_HEADER
- added U$1: RTL_SDR_CONN, mylib:RTL_SDR_CONN
Connections:
- net GND: now also JH1.P$4; no longer JP1.4
- net N$12: now also JH1.P$1; no longer JP1.1
- net N$4: now also JH1.P$2; no longer JP1.2
- net N$5: now also JH1.P$3; no longer JP1.3
Changed lines of the file:
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@@
 <part name="GND15" library="SparkFun-PowerSymbols" deviceset="GND" device=""/>
 <part name="GND24" library="SparkFun-PowerSymbols" deviceset="GND" device=""/>
-<part name="JP1" library="SparkFun-Connectors" deviceset="USB_SOLDER_PADS" device=""/>
 <part name="L6" library="mylib" deviceset="L_0805_PTH" device="" value="220uH"/>
 <part name="C8" library="mylib" deviceset="C_0805_PTH" device="" value="100nF"/>
 <part name="GND9" library="SparkFun-PowerSymbols" deviceset="GND" device=""/>
+<part name="U$1" library="mylib" deviceset="RTL_SDR_CONN" device=""/>
+<part name="JH1" library="mylib" deviceset="4X_PIN_HEADER" device=""/>
 </parts>
 <sheets>
@@
 <attribute name="VALUE" x="-22.86" y="139.446" size="1.778" layer="96" align="top-center"/>
 </instance>
-<instance part="JP1" gate="JP1" x="33.02" y="147.32" smashed="yes" rot="R180">
-<attribute name="VALUE" x="38.1" y="154.686" size="1.778" layer="96" font="vector" rot="R180"/>
-<attribute name="NAME" x="38.1" y="139.192" size="1.778" layer="95" font="vector" rot="R180"/>
-</instance>
 <instance part="L6" gate="L$1" x="17.78" y="162.56" smashed="yes" rot="R180">
 <attribute name="NAME" x="19.05" y="167.64" size="1.778" layer="95" rot="R270"/>
@@
 <attribute name="VALUE" x="35.814" y="175.26" size="1.778" layer="96" rot="R90" align="top-center"/>
 </instance>
+<instance part="U$1" gate="G$1" x="76.2" y="132.08" smashed="yes"/>
+<instance part="JH1" gate="G$1" x="30.48" y="149.86" smashed="yes"/>
 </instances>
 <busses>
@@
 <wire x1="17.78" y1="139.7" x2="17.78" y2="142.24" width="0.1524" layer="91"/>
 <wire x1="17.78" y1="142.24" x2="7.62" y2="142.24" width="0.1524" layer="91"/>
-<pinref part="JP1" gate="JP1" pin="4"/>
 <wire x1="27.94" y1="142.24" x2="17.78" y2="142.24" width="0.1524" layer="91"/>
 <junction x="17.78" y="142.24"/>
+<pinref part="JH1" gate="G$1" pin="P$4"/>
+<wire x1="30.48" y1="142.24" x2="27.94" y2="142.24" width="0.1524" layer="91"/>
 </segment>
 <segment>
@@
 <segment>
 <pinref part="J1" gate="G$1" pin="2"/>
-<pinref part="JP1" gate="JP1" pin="2"/>
 <wire x1="7.62" y1="147.32" x2="27.94" y2="147.32" width="0.1524" layer="91"/>
+<pinref part="JH1" gate="G$1" pin="P$2"/>
+<wire x1="30.48" y1="147.32" x2="27.94" y2="147.32" width="0.1524" layer="91"/>
 </segment>
 </net>
@@
 <segment>
 <pinref part="J1" gate="G$1" pin="3"/>
-<pinref part="JP1" gate="JP1" pin="3"/>
 <wire x1="7.62" y1="144.78" x2="27.94" y2="144.78" width="0.1524" layer="91"/>
+<pinref part="JH1" gate="G$1" pin="P$3"/>
+<wire x1="30.48" y1="144.78" x2="27.94" y2="144.78" width="0.1524" layer="91"/>
 </segment>
 </net>
@@
 <pinref part="J1" gate="G$1" pin="1"/>
 <wire x1="7.62" y1="149.86" x2="17.78" y2="149.86" width="0.1524" layer="91"/>
-<pinref part="JP1" gate="JP1" pin="1"/>
 <wire x1="27.94" y1="149.86" x2="17.78" y2="149.86" width="0.1524" layer="91"/>
 <pinref part="L6" gate="L$1" pin="1"/>
 <wire x1="17.78" y1="154.94" x2="17.78" y2="149.86" width="0.1524" layer="91"/>
 <junction x="17.78" y="149.86"/>
-</segment>
-</net>
+<pinref part="JH1" gate="G$1" pin="P$1"/>
+<wire x1="30.48" y1="149.86" x2="27.94" y2="149.86" width="0.1524" layer="91"/>
+</segment>
+</net>

Commit message: update
Parts:
- added C14: 56pF, mylib:C_0805_PTH
- added L7: 56nH, 164-11A06L:164-11A06L
- added L8: 82nH, 164-11A06L:164-11A06L
- added RF_OUT_VHF: 2X_SMD_PTH_PIN, mylib:2X_SMD_PTH_PIN
- C10: value 12pF -> 100pF
- C11: value 15pF -> 56pF
- C12: value 15pF -> 47pF
- C13: value 33pF -> 47pF
- C9: value 100pF -> 10nF
- L3: value 39nH -> 82nH; device mylib:L_0805_PTH -> 164-11A06L:164-11A06L
- L4, L5: value 39nH -> 56nH; device mylib:L_0805_PTH -> 164-11A06L:164-11A06L
Connections:
- new net N$14: C10.1, RF_OUT_VHF.PIN0
- new net N$19: C13.2, C14.1, L7.2
- net GND: now also L7.1, L8.1, RF_IN.PIN1, RF_OUT_VHF.PIN1; no longer C10.2, RF_IN.PIN0
- net N$10: now also RF_IN.PIN0; no longer RF_IN.PIN1
- net N$15: now also C9.1; no longer C10.1, C9.2
- net N$18: now also C10.2, C14.2, L8.2; no longer C13.2
- net N$2: now also C9.2; no longer C9.1
Other:
- moved on the sheet: C10, C11, C12, C13, C9, RF_IN

Commit message: update
Parts:
- removed L6: 220uH, mylib:L_0805_PTH
- removed RF_OUT_VHF: 2X_SMD_PTH_PIN, mylib:2X_SMD_PTH_PIN
- added C15, C16: 100nF, mylib:C_0805_PTH
- added C17: (no value), rcl:CPOL-EUE3.5-10
- added L10, L9: 220uH, mylib:L_0805_PTH
- added RF_IN_VHF: 2X_SMD_PTH_PIN, mylib:2X_SMD_PTH_PIN
Connections:
- removed net N$14: C10.1, RF_OUT_VHF.PIN0
- new net N$20: JH1.P$4, L9.1
- new net N$21: JH1.P$1, L10.2
- net GND: now also C15.1, C16.1, C17.-, L9.2, RF_IN_VHF.PIN0, RF_OUT.PIN1; no longer JH1.P$4, RF_OUT.PIN0, RF_OUT_VHF.PIN1
- net N$12: now also C10.1, RF_IN_VHF.PIN1; no longer J1.1, JH1.P$1, L6.1
- net N$18: now also RF_OUT.PIN0; no longer RF_OUT.PIN1
- net VCC: now also C15.2, C16.2, C17.+, J1.1, L10.1; no longer L6.2
Other:
- moved on the sheet: C8, RF_OUT

Commit message: Update
Parts:
- C2: value 100pF -> 22pF
- C3: value 200pF -> 150pF
- C4: value 100pF -> 150pF
Changed lines of the file:
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@@
 <part name="GND3" library="SparkFun-PowerSymbols" deviceset="GND" device=""/>
 <part name="C1" library="mylib" deviceset="C_0805_PTH" device="" value="100nF"/>
-<part name="C2" library="mylib" deviceset="C_0805_PTH" device="" value="100pF"/>
+<part name="C2" library="mylib" deviceset="C_0805_PTH" device="" value="22pF"/>
 <part name="GND4" library="SparkFun-PowerSymbols" deviceset="GND" device=""/>
 <part name="L1" library="mylib" deviceset="L_0805_PTH" device=""/>
 <part name="L2" library="mylib" deviceset="L_0805_PTH" device=""/>
-<part name="C3" library="mylib" deviceset="C_0805_PTH" device="" value="200pF"/>
+<part name="C3" library="mylib" deviceset="C_0805_PTH" device="" value="150pF"/>
 <part name="GND5" library="SparkFun-PowerSymbols" deviceset="GND" device=""/>
-<part name="C4" library="mylib" deviceset="C_0805_PTH" device="" value="100pF"/>
+<part name="C4" library="mylib" deviceset="C_0805_PTH" device="" value="150pF"/>
 <part name="GND6" library="SparkFun-PowerSymbols" deviceset="GND" device=""/>
 <part name="C5" library="mylib" deviceset="C_0805_PTH" device="" value="100nF"/>
