File: projects/RADIO/LNAs/tester_board/tester_board.sch (EAGLE design)
At the start: 6 parts, among them X1 SMA-142-0711-821/826

Commit message: update
Parts:
- removed X2: (no value), con-wago-500:W237-102
- added CON1: CON_SCREW_CLAMP_7MM, mylib:CON_SCREW_CLAMP_7MM
- added SMA-1: SMA_TH, mylib:SMA_TH
Connections:
- net GND: now also CON1G$2.1, SMA-1.GND@1; no longer X2-1.KL
- net N$1: now also CON1G$1.1, SMA-1.1; no longer X2-2.KL
Changed lines of the file:
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@@
 <parts>
 <part name="X1" library="con-coax" library_urn="urn:adsk.eagle:library:133" deviceset="SMA-" device="142-0711-821/826" package3d_urn="urn:adsk.eagle:package:6224/1"/>
-<part name="X2" library="con-wago-500" library_urn="urn:adsk.eagle:library:195" deviceset="W237-102" device="" package3d_urn="urn:adsk.eagle:package:10688/1"/>
 <part name="GND1" library="SparkFun-PowerSymbols" deviceset="GND" device=""/>
 <part name="GND2" library="SparkFun-PowerSymbols" deviceset="GND" device=""/>
@@
 <part name="GND5" library="SparkFun-PowerSymbols" deviceset="GND" device=""/>
 <part name="GND6" library="SparkFun-PowerSymbols" deviceset="GND" device=""/>
+<part name="CON1" library="mylib" deviceset="CON_SCREW_CLAMP_7MM" device=""/>
+<part name="SMA-1" library="mylib" deviceset="SMA_TH" device=""/>
+<part name="GND7" library="SparkFun-PowerSymbols" deviceset="GND" device=""/>
 </parts>
 <sheets>
@@
 <instance part="X1" gate="G1" x="17.78" y="60.96" smashed="yes">
 <attribute name="NAME" x="15.24" y="64.262" size="1.778" layer="95"/>
-</instance>
-<instance part="X2" gate="-1" x="55.88" y="55.88" smashed="yes" rot="R180">
-<attribute name="NAME" x="55.88" y="54.991" size="1.778" layer="95"/>
-</instance>
-<instance part="X2" gate="-2" x="55.88" y="60.96" smashed="yes" rot="R180">
-<attribute name="VALUE" x="58.42" y="64.643" size="1.778" layer="96" rot="R180"/>
-<attribute name="NAME" x="55.88" y="60.071" size="1.778" layer="95"/>
 </instance>
 <instance part="GND1" gate="1" x="22.86" y="50.8" smashed="yes">
@@
 <attribute name="VALUE" x="56.134" y="27.94" size="1.778" layer="96" rot="R90" align="top-center"/>
 </instance>
+<instance part="CON1" gate="G$1" x="60.96" y="60.96" smashed="yes">
+<attribute name="NAME" x="54.61" y="64.135" size="1.778" layer="95"/>
+<attribute name="VALUE" x="54.61" y="55.88" size="1.778" layer="96"/>
+</instance>
+<instance part="CON1" gate="G$2" x="60.96" y="55.88" smashed="yes">
+<attribute name="NAME" x="54.61" y="59.055" size="1.778" layer="95"/>
+<attribute name="VALUE" x="54.61" y="50.8" size="1.778" layer="96"/>
+</instance>
+<instance part="SMA-1" gate="G$1" x="7.62" y="60.96" smashed="yes">
+<attribute name="VALUE" x="5.08" y="53.34" size="1.778" layer="96"/>
+<attribute name="NAME" x="5.08" y="64.262" size="1.778" layer="95"/>
+</instance>
+<instance part="GND7" gate="1" x="10.16" y="50.8" smashed="yes">
+<attribute name="VALUE" x="10.16" y="50.546" size="1.778" layer="96" align="top-center"/>
+</instance>
 </instances>
 <busses>
@@
 <segment>
 <pinref part="X1" gate="G1" pin="1"/>
-<pinref part="X2" gate="-2" pin="KL"/>
-<wire x1="20.32" y1="60.96" x2="50.8" y2="60.96" width="0.1524" layer="91"/>
+<wire x1="20.32" y1="60.96" x2="25.4" y2="60.96" width="0.1524" layer="91"/>
+<pinref part="CON1" gate="G$1" pin="1"/>
+<wire x1="25.4" y1="60.96" x2="50.8" y2="60.96" width="0.1524" layer="91"/>
+<wire x1="58.42" y1="60.96" x2="50.8" y2="60.96" width="0.1524" layer="91"/>
+<pinref part="SMA-1" gate="G$1" pin="1"/>
+<wire x1="10.16" y1="60.96" x2="10.16" y2="68.58" width="0.1524" layer="91"/>
+<wire x1="10.16" y1="68.58" x2="25.4" y2="68.58" width="0.1524" layer="91"/>
+<wire x1="25.4" y1="68.58" x2="25.4" y2="60.96" width="0.1524" layer="91"/>
+<junction x="25.4" y="60.96"/>
 </segment>
 </net>
@@
 <segment>
 <pinref part="GND2" gate="1" pin="GND"/>
-<pinref part="X2" gate="-1" pin="KL"/>
 <wire x1="45.72" y1="53.34" x2="45.72" y2="55.88" width="0.1524" layer="91"/>
 <wire x1="45.72" y1="55.88" x2="50.8" y2="55.88" width="0.1524" layer="91"/>
+<pinref part="CON1" gate="G$2" pin="1"/>
+<wire x1="58.42" y1="55.88" x2="50.8" y2="55.88" width="0.1524" layer="91"/>
 </segment>
 <segment>
@@
 <wire x1="53.34" y1="27.94" x2="48.26" y2="27.94" width="0.1524" layer="91"/>
 </segment>
+<segment>
+<pinref part="GND7" gate="1" pin="GND"/>
+<pinref part="SMA-1" gate="G$1" pin="GND@1"/>
+<wire x1="10.16" y1="53.34" x2="10.16" y2="58.42" width="0.1524" layer="91"/>
+</segment>
 </net>
